File: hardware/bridge.kicad_sch (KiCad schematic)
At the start: 67 parts, among them J2 MOTOR, Q1 TPN1R603PL, Q2 TPN1R603PL, Q3 TPN1R603PL, Q4 TPN1R603PL, Q5 TPN1R603PL, Q6 TPN1R603PL, Q7 TPN1R603PL, Q8 TPN1R603PL

Commit message: Rev 0.2: 内蔵機能 (電流源/シンク・USB-PD・OPA/CMP 全モード) の活用
回路 (102/102 ネット一致):
- USB-PD シンクでモーター電源を供給: F3 → U5 LM74700 + Q10 → VBUS (PC3 で許可),
  USB VBUS 監視 (PA2), SMAJ20A。USBLC6 の基準を +3V3 に変更 (VBUS 20V 対策)
- J1 の逆接保護を U4 LM74700 + Q9 のハイサイド理想ダイオードに変更 (J1 / PD を安全に OR)
- 3 相センシングを PA5/PA6/PA7 に集約 (W 相 PA12 → PA6): CMP3 内部仮想中性点 + TIM2 捕捉
  によるセンサレス BEMF 検出, TIM2 ホール XOR, ISOURCE2 結線診断を同じピンで利用
- JP7: OPA3 入力を HB0 レッグ / バス電流で切替 (CMP2 + DAC でバス過電流・電流制限)
- JP8 + C105: QII1 (OPA1 → CMP1 → TIM3) でタコ / VR センサ / ブラシ DC 電流リップル計数
- 状態 LED を PC4 (USER/BOOT) と共用, J6/J7 を再割当 (1 線 SDI)

ファームウェア (警告 0):
- mpb.h ライブラリ: PD シンク (WCH USBPD_SNK 移植 + 8〜15V ポリシー + 給電パス制御),
  過電流保護 (CMP3/CMP2+DAC, TIM2 停止割込み), BEMF, ホール, タコ, NTC, 結線自己診断, TIM3 時間基準
- ブートローダ / テンプレートの状態 LED を PC4 (オープンドレイン) に変更

ドキュメント: docs/advanced_features.md (検討と判断, 要実機確認事項, Rev 0.3 候補)

Co-Authored-By: Claude Opus 5.5 <noreply@anthropic.com>
Claude-Session: https://claude.ai/code/session_01LENFjjhDfYjJZV1NWhB9uV
Parts:
- added JP7: ISEL_A, Connector_PinHeader_2.54mm:PinHeader_1x03_P2.54mm_Vertical, symbol mdrv:CONN3
- JP5: value ISEL -> ISEL_B
Connections:
- net ISH: now also JP7.3 (P3)
- net SRC0: now also JP7.1 (P1)
- new net ISA_SEL: JP7.2 (P2)
Other:
- note added: "JP7 1-2: ISP1=HB0 (差動) 2-3: ISP1=バス (ISH, OPA3 を単端 NSEL=VSS で使用)"
- note added: "RS_BUS(R70) は全レッグ共通の帰路 → PB3 で ADC 計測 + CMP3 過電流ブレーキ, JP8 経由で QII1 (リップル)"
- note added: "ホール: 同じ 3 ピンが TIM2 CH1-3 → ホールセンサ XOR モードでハード計時。ISOURCE2/ISINK も同ピン (結線自己診断)。"
- note added: "分圧比 3/23。センサレス: CMP3 が各相 (N) を内部仮想中性点 (RMID, 80k x3) と比較し TIM2 でゼロクロス時刻を捕捉。"
- note added: "相電圧 (BEMF) / ホール 切替 → PA5/PA6/PA7 (CMP3 N0-N2 = TIM2 CH1-3)"
- note removed: "RS_BUS(R70) は全レッグ共通の帰路 → PB3 で ADC 計測 + CMP3 過電流ブレーキ"
- note removed: "ジャンパ未実装時は SENS_x (PA5/PA7/PA12) を汎用 GPIO/ADC として JP 中央ピンから利用可。"
- note removed: "分圧比 3/23: VBUS 16V → 2.09V。センサレスは ADC で相電圧を PWM ON 中に標本化 (VBUS/2 比較)。"
- note removed: "相電圧 (BEMF) 検出 / ホール・相電圧 切替"
Changed lines of the file:
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@@
 (kicad_sch (version 20230121) (generator eeschema)
 (paper "A3")
-(title_block (title "mPBCH32M030DS0  CH32M030 Universal Motor Driver") (date "2026-09-24") (rev "0.1") (company "ghostinkoma") (comment 1 "パワー段 (4 ハーフブリッジ) / ゲート確認 LED / シャント / モータ出力") (comment 2 "個人利用可 (クレジット表示必須) / 商用利用は要連絡 / 無保証  -  LICENSE 参照"))
+(title_block (title "mPBCH32M030DS0  CH32M030 Universal Motor Driver") (date "2026-09-24") (rev "0.2") (company "ghostinkoma") (comment 1 "パワー段 (4 ハーフブリッジ) / ゲート確認 LED / シャント / モータ出力") (comment 2 "個人利用可 (クレジット表示必須) / 商用利用は要連絡 / 無保証  -  LICENSE 参照"))
 (rectangle (start 15 20) (end 109 142) (stroke (width 0.2) (type dash)) (fill (type none)))
 (text "ハーフブリッジ HB0  (OUT0)" (at 17 25 0) (effects (font (size 2 2) (thickness 0.3) bold) (justify left bottom)))
@@
 (text "バスシャント / 電流チャネル選択 / モータ端子" (at 17 155 0) (effects (font (size 2 2) (thickness 0.3) bold) (justify left bottom)))
 (rectangle (start 155 150) (end 405 240) (stroke (width 0.2) (type dash)) (fill (type none)))
-(text "相電圧 (BEMF) 検出 / ホール・相電圧 切替" (at 157 155 0) (effects (font (size 2 2) (thickness 0.3) bold) (justify left bottom)))
+(text "相電圧 (BEMF) / ホール 切替 → PA5/PA6/PA7 (CMP3 N0-N2 = TIM2 CH1-3)" (at 157 155 0) (effects (font (size 2 2) (thickness 0.3) bold) (justify left bottom)))
 (text "ゲート: 47Ω 直列 + 20kΩ G-S プルダウン (WCH 評価ボード準拠)。シャント 10mΩ はケルビン接続。" (at 18 138 0) (effects (font (size 1.3 1.3)) (justify left bottom)))
 (text "J2: 3相=U/V/W(1-3) | DC=1-2 (+3-4) | ステッピング=A+,A-,B+,B-" (at 20 255 0) (effects (font (size 1.4 1.4)) (justify left bottom)))
 (text "JP5 1-2: ISP2=HB1(V相)  2-3: ISP2=HB2(コイルB / DC-B)" (at 20 262 0) (effects (font (size 1.4 1.4)) (justify left bottom)))
-(text "RS_BUS(R70) は全レッグ共通の帰路 → PB3 で ADC 計測 + CMP3 過電流ブレーキ" (at 20 269 0) (effects (font (size 1.4 1.4)) (justify left bottom)))
-(text "分圧比 3/23: VBUS 16V → 2.09V。センサレスは ADC で相電圧を PWM ON 中に標本化 (VBUS/2 比較)。" (at 160 228 0) (effects (font (size 1.3 1.3)) (justify left bottom)))
-(text "ジャンパ未実装時は SENS_x (PA5/PA7/PA12) を汎用 GPIO/ADC として JP 中央ピンから利用可。" (at 160 234 0) (effects (font (size 1.3 1.3)) (justify left bottom)))
+(text "JP7 1-2: ISP1=HB0 (差動)  2-3: ISP1=バス (ISH, OPA3 を単端 NSEL=VSS で使用)" (at 20 248 0) (effects (font (size 1.4 1.4)) (justify left bottom)))
+(text "RS_BUS(R70) は全レッグ共通の帰路 → PB3 で ADC 計測 + CMP3 過電流ブレーキ, JP8 経由で QII1 (リップル)" (at 20 269 0) (effects (font (size 1.4 1.4)) (justify left bottom)))
+(text "分圧比 3/23。センサレス: CMP3 が各相 (N) を内部仮想中性点 (RMID, 80k x3) と比較し TIM2 でゼロクロス時刻を捕捉。" (at 160 228 0) (effects (font (size 1.3 1.3)) (justify left bottom)))
+(text "ホール: 同じ 3 ピンが TIM2 CH1-3 → ホールセンサ XOR モードでハード計時。ISOURCE2/ISINK も同ピン (結線自己診断)。" (at 160 234 0) (effects (font (size 1.3 1.3)) (justify left bottom)))
 (symbol (lib_id "mdrv:NMOS") (at 60.72 50.8 0) (unit 1) (in_bom yes) (on_board yes) (dnp no)
 (property "Reference" "Q1" (at 64.53 49.53 0) (effects (font (size 1.27 1.27)) (justify left)))
@@
 (global_label "VBUS" (shape passive) (at 83.58 64.77 90) (fields_autoplaced) (effects (font (size 1.27 1.27)) (justify left)) (property "Intersheetrefs" "${INTERSHEET_REFS}" (at 83.58 64.77 0) (effects (font (size 1.27 1.27)) hide)))
 (wire (pts (xy 83.58 74.93) (xy 83.58 77.47)) (stroke (width 0) (type default)))
-(global_label "SRC0" (shape passive) (at 83.58 77.47 270) (fields_autoplaced) (effects (font (size 1.27 1.27)) (justify right)) (property "Intersheetrefs" "${INTERSHEET_REFS}" (at 83.58 77.47 0) (effects (font (size 1.27 1.27)) hide)))
+(label "SRC0" (at 83.58 77.47 270) (fields_autoplaced) (effects (font (size 1.27 1.27)) (justify right bottom)))
 (symbol (lib_id "mdrv:C") (at 96.28 71.12 0) (unit 1) (in_bom yes) (on_board yes) (dnp no)
 (property "Reference" "C31" (at 98.82 69.85 0) (effects (font (size 1.27 1.27)) (justify left)))
@@
 (global_label "VBUS" (shape passive) (at 96.28 64.77 90) (fields_autoplaced) (effects (font (size 1.27 1.27)) (justify left)) (property "Intersheetrefs" "${INTERSHEET_REFS}" (at 96.28 64.77 0) (effects (font (size 1.27 1.27)) hide)))
 (wire (pts (xy 96.28 74.93) (xy 96.28 77.47)) (stroke (width 0) (type default)))
-(global_label "SRC0" (shape passive) (at 96.28 77.47 270) (fields_autoplaced) (effects (font (size 1.27 1.27)) (justify right)) (property "Intersheetrefs" "${INTERSHEET_REFS}" (at 96.28 77.47 0) (effects (font (size 1.27 1.27)) hide)))
+(label "SRC0" (at 96.28 77.47 270) (fields_autoplaced) (effects (font (size 1.27 1.27)) (justify right bottom)))
 (symbol (lib_id "mdrv:R") (at 78.72 120.44 90) (unit 1) (in_bom yes) (on_board yes) (dnp no)
 (property "Reference" "R35" (at 78.72 117.64 90) (effects (font (size 1.27 1.27))))
@@
 )
 (wire (pts (xy 94.53 130.44) (xy 97.07 130.44)) (stroke (width 0) (type default)))
-(global_label "SRC0" (shape passive) (at 97.07 130.44 0) (fields_autoplaced) (effects (font (size 1.27 1.27)) (justify left)) (property "Intersheetrefs" "${INTERSHEET_REFS}" (at 97.07 130.44 0) (effects (font (size 1.27 1.27)) hide)))
+(label "SRC0" (at 97.07 130.44 0) (fields_autoplaced) (effects (font (size 1.27 1.27)) (justify left bottom)))
 (symbol (lib_id "mdrv:NMOS") (at 158.72 50.8 0) (unit 1) (in_bom yes) (on_board yes) (dnp no)
 (property "Reference" "Q3" (at 162.53 49.53 0) (effects (font (size 1.27 1.27)) (justify left)))
@@
 (symbol (lib_id "mdrv:CONN3") (at 45 195 0) (unit 1) (in_bom yes) (on_board yes) (dnp no)
 (property "Reference" "JP5" (at 45 192.46 0) (effects (font (size 1.27 1.27)) (justify left)))
-(property "Value" "ISEL" (at 45 189.92 0) (effects (font (size 1.27 1.27)) (justify left)))
+(property "Value" "ISEL_B" (at 45 189.92 0) (effects (font (size 1.27 1.27)) (justify left)))
 (property "Footprint" "Connector_PinHeader_2.54mm:PinHeader_1x03_P2.54mm_Vertical" (at 45 195 0) (effects (font (size 1.27 1.27)) hide))
 (property "Datasheet" "~" (at 45 195 0) (effects (font (size 1.27 1.27)) hide))
@@
 (wire (pts (xy 39.92 200.08) (xy 37.38 200.08)) (stroke (width 0) (type default)))
 (label "SRC2" (at 37.38 200.08 180) (fields_autoplaced) (effects (font (size 1.27 1.27)) (justify right bottom)))
+(symbol (lib_id "mdrv:CONN3") (at 45 225 0) (unit 1) (in_bom yes) (on_board yes) (dnp no)
+(property "Reference" "JP7" (at 45 222.46 0) (effects (font (size 1.27 1.27)) (justify left)))
+(property "Value" "ISEL_A" (at 45 219.92 0) (effects (font (size 1.27 1.27)) (justify left)))
+(property "Footprint" "Connector_PinHeader_2.54mm:PinHeader_1x03_P2.54mm_Vertical" (at 45 225 0) (effects (font (size 1.27 1.27)) hide))
+(property "Datasheet" "~" (at 45 225 0) (effects (font (size 1.27 1.27)) hide))
+(property "MPN" "2.54mm 3P + ジャンパ (1-2: HB0 レッグ / 2-3: バス電流)" (at 45 225 0) (effects (font (size 1.27 1.27)) hide))
+(pin "1")
+(pin "2")
+(pin "3")
+(instances (project "mPBCH32M030DS0" (path "/cb038f79-02b6-58e4-b0e9-4ee93e4d05b7/438ea180-5cfc-5f9d-8f47-84e352028664" (reference "JP7") (unit 1))))
+)
+(wire (pts (xy 39.92 225) (xy 37.38 225)) (stroke (width 0) (type default)))
+(label "SRC0" (at 37.38 225 180) (fields_autoplaced) (effects (font (size 1.27 1.27)) (justify right bottom)))
+(wire (pts (xy 39.92 227.54) (xy 37.38 227.54)) (stroke (width 0) (type default)))
+(global_label "ISA_SEL" (shape passive) (at 37.38 227.54 180) (fields_autoplaced) (effects (font (size 1.27 1.27)) (justify right)) (property "Intersheetrefs" "${INTERSHEET_REFS}" (at 37.38 227.54 0) (effects (font (size 1.27 1.27)) hide)))
+(wire (pts (xy 39.92 230.08) (xy 37.38 230.08)) (stroke (width 0) (type default)))
+(global_label "ISH" (shape passive) (at 37.38 230.08 180) (fields_autoplaced) (effects (font (size 1.27 1.27)) (justify right)) (property "Intersheetrefs" "${INTERSHEET_REFS}" (at 37.38 230.08 0) (effects (font (size 1.27 1.27)) hide)))
 (symbol (lib_id "mdrv:CONN4") (at 110 175 0) (unit 1) (in_bom yes) (on_board yes) (dnp no)
 (property "Reference" "J2" (at 110 172.46 0) (effects (font (size 1.27 1.27)) (justify left)))
@@
 (global_label "SW0" (shape passive) (at 73.42 71.12 0) (fields_autoplaced) (effects (font (size 1.27 1.27)) (justify left)) (property "Intersheetrefs" "${INTERSHEET_REFS}" (at 73.42 71.12 0) (effects (font (size 1.27 1.27)) hide)))
 (label "GL0" (at 51.83 88.9 90) (fields_autoplaced) (effects (font (size 1.27 1.27)) (justify left bottom)))
-(global_label "SRC0" (shape passive) (at 73.42 104.14 0) (fields_autoplaced) (effects (font (size 1.27 1.27)) (justify left)) (property "Intersheetrefs" "${INTERSHEET_REFS}" (at 73.42 104.14 0) (effects (font (size 1.27 1.27)) hide)))
+(label "SRC0" (at 73.42 104.14 0) (fields_autoplaced) (effects (font (size 1.27 1.27)) (justify left bottom)))
 (global_label "VBUS" (shape passive) (at 158.72 43.18 90) (fields_autoplaced) (effects (font (size 1.27 1.27)) (justify left)) (property "Intersheetrefs" "${INTERSHEET_REFS}" (at 158.72 43.18 0) (effects (font (size 1.27 1.27)) hide)))
 (label "GH1" (at 149.83 48.26 90) (fields_autoplaced) (effects (font (size 1.27 1.27)) (justify left bottom)))
