File: hardware/mcu.kicad_sch (KiCad schematic)
At the start: 25 parts, among them U1 CH32M030C8U7

Commit message: Rev 0.2: 内蔵機能 (電流源/シンク・USB-PD・OPA/CMP 全モード) の活用
回路 (102/102 ネット一致):
- USB-PD シンクでモーター電源を供給: F3 → U5 LM74700 + Q10 → VBUS (PC3 で許可),
  USB VBUS 監視 (PA2), SMAJ20A。USBLC6 の基準を +3V3 に変更 (VBUS 20V 対策)
- J1 の逆接保護を U4 LM74700 + Q9 のハイサイド理想ダイオードに変更 (J1 / PD を安全に OR)
- 3 相センシングを PA5/PA6/PA7 に集約 (W 相 PA12 → PA6): CMP3 内部仮想中性点 + TIM2 捕捉
  によるセンサレス BEMF 検出, TIM2 ホール XOR, ISOURCE2 結線診断を同じピンで利用
- JP7: OPA3 入力を HB0 レッグ / バス電流で切替 (CMP2 + DAC でバス過電流・電流制限)
- JP8 + C105: QII1 (OPA1 → CMP1 → TIM3) でタコ / VR センサ / ブラシ DC 電流リップル計数
- 状態 LED を PC4 (USER/BOOT) と共用, J6/J7 を再割当 (1 線 SDI)

ファームウェア (警告 0):
- mpb.h ライブラリ: PD シンク (WCH USBPD_SNK 移植 + 8〜15V ポリシー + 給電パス制御),
  過電流保護 (CMP3/CMP2+DAC, TIM2 停止割込み), BEMF, ホール, タコ, NTC, 結線自己診断, TIM3 時間基準
- ブートローダ / テンプレートの状態 LED を PC4 (オープンドレイン) に変更

ドキュメント: docs/advanced_features.md (検討と判断, 要実機確認事項, Rev 0.3 候補)

Co-Authored-By: Claude Opus 5.5 <noreply@anthropic.com>
Claude-Session: https://claude.ai/code/session_01LENFjjhDfYjJZV1NWhB9uV
Connections:
- net GPIO_PA6 is gone; now on net SENS_W: U1.43 (PA6/CM3N1/T2C2/ISINK1)
- net SENS_W: no longer U1.1 (PA12/QII1/A19)
- net GPIO_PC3 renamed PD_PWR_EN
- net SRC0 renamed ISA_SEL
- net SWCLK renamed USB_VBUS_SNS
- new net QII_IN: U1.1 (PA12/QII1(OPA1)/A19)
Other:
- note added: "3 相センシング PA5/PA6/PA7 = CMP3 N0/N1/N2 (内部仮想中性点 RMID + TIM2 キャプチャ) = TIM2 CH1/2/3 (ホール XOR)"
- note added: "CMP2: P=OPA3 出力, N=内蔵 DAC (0.1〜3.1V/0.2V) → TIM1 BKIN (サイクル毎電流制限にも)。"
- note added: "CMP3 → TIM1 BKIN。センサレス (CMP3 を BEMF 用に使う) 時は JP7=バスにして CMP2 で遮断。"
- note added: "I2C: PA14/PA15 (リマップ2)。UART: PC1/PC2 (リマップ1)。RST: PC0。SDI 1 線: PA3。水晶: PB5/PB6"
- note added: "J6 引き出し: PC4 (USER/BOOT + 状態 LED), PC5 (HV I/O), TACH_IN, nFAULT (PA13 = TIM1_BKIN_1)"
- note added: "PWM: HB0〜HB2 = TIM1 (相補+ブレーキ)。HB2/HB3 を TIM2 リマップ2 (PB12〜PB15) で駆動すれば 4 レッグ全て相補"
- note added: "QII1: PA12 → OPA1 (AV20/40) → CMP1 → TIM3 CH1 キャプチャ (JP8: タコ/VR 入力 or バス電流リップル)"
- note added: "USB: CC1/CC2 = PA0/PA1 (PD0 シンク), D+/D- = PB0/PB1, USB VBUS 監視 = PA2, PD 給電許可 = PC3"
- note added: "保護: CMP3 (PB3 vs PB2) または CMP2 (OPA3 出力 vs 内蔵 DAC) → TIM1 BKIN。PB4 OVP リセット"
- note added: "電流: IA = OPA3 (JP7: HB0 レッグ / バス) → ADC9, IB = OPA4 (JP5: HB1 / HB2) → ADC10, IBUS = PB3 直接 → ADC1"
- note added: "電流アンプ入力 (OPA3=ISP1: JP7 選択 / OPA4=ISP2: JP5 選択 → ADC 内部接続)"
- note removed: "(DS 1.4.20: 2 組のフルブリッジは PB8〜PB11 = TIM1, PB12〜PB15 = TIM2 で駆動) → 4 レッグ全て相補 PWM"
- note removed: "CMP2: P=OPA3 出力, N=DAC1 → TIM1 BKIN (HB0 レッグの第2過電流保護)。"
- note removed: "CMP3 → TIM1 BKIN (ハード遮断)。TIM2 (HB2/HB3 を TIM2 駆動時) は CMP3 割込みで FW 停止。"
- note removed: "HB0〜HB2: TIM1 CH1/CH1N〜CH3/CH3N (デフォルト配置)。TIM1 リマップ1 で BKIN を PA13 (nFAULT) へ"
- note removed: "HB2/HB3 を TIM2 で駆動する場合: TIM2 リマップ2 → PB13/PB12 = CH1/CH1N, PB15/PB14 = CH2/CH2N"
- note removed: "I2C: PA14/PA15 (I2C リマップ2)。UART: PC1=TX / PC2=RX (UART リマップ1)"
- note removed: "USB: PA0/PA1 = CC1/CC2, PB0/PB1 = D+/D-。水晶: PB5/PB6。RST: PC0。SWD: PA2/PA3"
- note removed: "センサ: SENS_U/V/W = PA5/PA7/PA12 (ADC_IN6/IN2/IN19 + EXTI)。JP2〜JP4 でホール/相電圧を選択"
- note removed: "相電流アンプ入力 (OPA3=ISP1 / OPA4=ISP2 差動 → ADC 内部接続)"
- note removed: "空き GPIO → J6: PC3, PC4 (USER/BOOT), PC5 (HV I/O, VHV レベル), PA6 (状態 LED 兼用)"
- note removed: "電流: IA (OPA3, HB0) / IB (OPA4, JP5 で HB1 or HB2) / IBUS (PB3 直接 ADC) を内蔵 ADC で計測"

Commit message: Rev 0.3: パワー段を子基板化 (A/B/C/D) し 2 層基板レイアウトを作成
構成:
- 主基板 (60x42mm, 2 層): 右 = CH32M030 / USB-C / GPIO・I2C・UART・SDI・HALL,
  左上 = 電源 (J1 → F1 → 理想ダイオード, USB-PD 経路), 左下 = 基板間コネクタ J9/J10 (裏面)
- 子基板と裏面同士を背中合わせに重ねる (基板間 約5mm, 裏面部品は高さ 2mm 以下)。
  RESET / USER・BOOT / センシング選択は主基板 TOP、電流チャネル選択 JP5/JP7 は子基板 TOP
- 子基板 A: TPN1R603PL (既存回路) / B: TKR74F04PB (24V 系, 66x66mm) /
  C: MTN2306AN3 (廉価版) / D: MOSFET なし (全信号をピンヘッダへ引き出し)
- 基板間ピンは同じ番号同士が嵌合 (ソケットを 270° 回転して裏面実装, 座標で全 32 ピンを検証)
- コネクタは USB-C 以外すべて 2.54mm ピンヘッダ。コンデンサは 1005/1608 基本
  (入手性を確認した量産品番。50V/10uF のみ 2012)
- 24V 対応: Q9 を 40V 品 (TPN2R304PL), VHV に 47Ω + 27V ツェナー, D1/R11 の 24V 用定数を注記,
  FW は make POWER_STAGE=B で VBUS 分圧比を切替
- F1 を NANO2 10A (SMD), スイッチを B3U-1000P に小型化

基板生成 (hardware/gen_pcb.py + pcblib.py):
- 配置 → Freerouting 1.9 自動配線 → 大電流ネットのベタ化 → GND ベタ・スティッチング
  → 残り接続の補修 (格子 A*, DRC が増えない経路のみ採用) → DRC
- 5 基板とも未接続 0・電気的 DRC エラー 0 (警告はシルクの重なりのみ)
- 製造データ hardware/fab/*.zip (ガーバー, ドリル, 両面の部品座標)

回路図: 主基板 82/82, 子基板 A/B/C 41/41, D 21/21 ネット一致。FW は A/B とも警告 0 でビルド。

Co-Authored-By: Claude Opus 5.5 <noreply@anthropic.com>
Claude-Session: https://claude.ai/code/session_01LENFjjhDfYjJZV1NWhB9uV
Parts:
- C10: footprint Capacitor_SMD:C_1210_3225Metric -> Capacitor_SMD:C_0805_2012Metric; MPN (none) -> TDK C2012X5R1H106K125AC (X5R 2012) ※50V/10uF は 1608 の量産品なし
- C11: footprint Capacitor_SMD:C_0603_1608Metric -> Capacitor_SMD:C_0402_1005Metric; MPN (none) -> Murata GRM155R71H104KE14D (X7R 1005)
- C12: footprint Capacitor_SMD:C_0805_2012Metric -> Capacitor_SMD:C_0603_1608Metric; MPN (none) -> Murata GRM188R61E106MA73D (X5R 1608)
- C13: value 0.1uF/25V -> 0.1uF/50V; footprint Capacitor_SMD:C_0603_1608Metric -> Capacitor_SMD:C_0402_1005Metric; MPN (none) -> Murata GRM155R71H104KE14D (X7R 1005)
- C14: MPN (none) -> Murata GRM155R61A475MEAAD (X5R 1005)
- C15: value 0.1uF/10V -> 0.1uF/50V; MPN (none) -> Murata GRM155R71H104KE14D (X7R 1005)
- C16: value 10nF -> 10nF/50V; MPN (none) -> Murata GRM155R71H103KA88D (X7R 1005)
- C17: MPN (none) -> Murata GRM1555C1H102JA01D (C0G 1005)
- C18: value 0.1uF -> 0.1uF/50V; MPN (none) -> Murata GRM155R71H104KE14D (X7R 1005)
- C19, C20: MPN (none) -> Murata GRM1555C1H222JA01D (C0G 1005)
- C21, C22, C23, C24: value 1uF/25V X7R -> 2.2uF/25V; footprint Capacitor_SMD:C_0805_2012Metric -> Capacitor_SMD:C_0603_1608Metric; MPN (none) -> Murata GRM188R61E225KA12D (X5R 1608)
- R11: MPN (none) -> 24V 系は 180k 1%
Other:
- note added: "2.2uF (1608, DC バイアス後 ≈1.3uF): Qg 41nC (A) で降下 32mV, Qg ≈150nC (B) でも ≈0.12V。"
- note added: "3 相センシング PA5/PA6/PA7 = CMP3 N0/N1/N2 (仮想中性点 + TIM2 キャプチャ) = TIM2 CH1/2/3 (ホール XOR)"
- note added: "CMP2: P=OPA3 出力, N=内蔵 DAC (0.1〜3.1V/0.2V) → TIM1 BKIN。"
- note added: "ISH / ISA_SEL / ISB_SEL は子基板のシャントから J10 経由で来る (ケルビン配線)。"
- note added: "OPA3 出力 → ADC_IN9, OPA4 出力 → ADC_IN10 (チップ内部接続)。電流チャネル選択 JP5/JP7 は子基板。"
- note added: "PB4: VBUS/12 → ADC_IN17 + OVP リセット (1.5V → 18.0V)。24V 系は R11=180k (VBUS/19, 28.5V)。"
- note added: "VHV 5〜28V (≥10uF)。VDD8 は FW で 5/8/9/10V 選択 (≥10uF)。VDD33 は 1〜10uF (DS 1.4.3)。"
- note added: "ブートストラップ容量 (VBx-VSx, MCU ピン直近 = 主基板)"
- note added: "電流: IA = OPA3 (子基板 JP7: HB0 / バス) → ADC9, IB = OPA4 (子基板 JP5: HB1 / HB2) → ADC10, IBUS = PB3"
- note added: "電流アンプ入力 (OPA3=ISP1 / OPA4=ISP2 → ADC 内部接続)"
- note removed: "3 相センシング PA5/PA6/PA7 = CMP3 N0/N1/N2 (内部仮想中性点 RMID + TIM2 キャプチャ) = TIM2 CH1/2/3 (ホール XOR)"
- note removed: "CMP2: P=OPA3 出力, N=内蔵 DAC (0.1〜3.1V/0.2V) → TIM1 BKIN (サイクル毎電流制限にも)。"
- note removed: "CMP3 → TIM1 BKIN。センサレス (CMP3 を BEMF 用に使う) 時は JP7=バスにして CMP2 で遮断。"
- note removed: "OPA3 出力 → ADC_IN9, OPA4 出力 → ADC_IN10 (チップ内部接続, RM 17.2.2)。"
- note removed: "PB4: VBUS/12 → ADC_IN17 + OVP リセット (1.5V → VBUS 18.0V で MCU リセット = 全ゲート OFF)。"
- note removed: "Qg=41nC に対し 1uF → 1 周期の電圧降下 ≈ 41mV。"
- note removed: "VHV 4.0〜29V (≥10uF)。VDD8 は FW で 5/8/9/10V 選択 (≥10uF)。VDD33 は 1〜10uF (DS 1.4.3)。"
- note removed: "ブートストラップ容量 (VBx-VSx, ピン直近)"
- note removed: "電流: IA = OPA3 (JP7: HB0 レッグ / バス) → ADC9, IB = OPA4 (JP5: HB1 / HB2) → ADC10, IBUS = PB3 直接 → ADC1"
- note removed: "電流アンプ入力 (OPA3=ISP1: JP7 選択 / OPA4=ISP2: JP5 選択 → ADC 内部接続)"
- title: mPBCH32M030DS0  CH32M030 Universal Motor Driver -> mPBCH32M030DS0  CH32M030 Universal Motor Driver - Main board

Commit message: Rev 0.4: DIP-42 MCU module + power boards A/B/C (KiCad 8)
- MCU module: 20.32 x 53.34mm (8 x 21 grid), DIP-42 (0.6in rows), fits
  an 82 x 52mm breadboard. Headers can be fitted from either side;
  signal names on bottom silk. All LEDs (power, status, 8 gate LEDs) on
  the module top.
- Power boards take the module in two 1x21 sockets (left/right
  symmetric mating). FETs/shunts on the heatsink side, no LEDs.
  Voltage-dependent parts (TVS, OVP divider, bulk caps, BEMF divider)
  moved to the power boards. Breakout board D removed.
  A/C: 20.32 x 71.94mm, B (TO-263 x8): 40.64 x 66.94mm.
- Capacitors re-selected for realistic size vs voltage/capacitance
  (4.7uF 1608, 10uF/25V 2012, 10uF/50V 1206, 4.7nF/100V 1608, low
  profile electrolytics).
- Schematics and boards generated in KiCad 8 format; netlists verified
  with KiCad 8.0.9.
- Layout pipeline: Freerouting bridge (parallel), second pass, early
  repair before pours, island-aware maze repair, DRC via kicad-cli.
- DRC: power boards A/B/C have 0 unconnected / 0 electrical errors.
  The MCU module still has unrouted connections (work in progress).

Co-Authored-By: Claude Opus 5.5 <noreply@anthropic.com>
Claude-Session: https://claude.ai/code/session_01LENFjjhDfYjJZV1NWhB9uV
Parts:
- removed C21, C22, C23, C24: 2.2uF/25V, Capacitor_SMD:C_0603_1608Metric, symbol mdrv:C
- added C10: 10uF/50V, Capacitor_SMD:C_1206_3216Metric, symbol mdrv:C
- added C11: 0.1uF/50V, Capacitor_SMD:C_0402_1005Metric, symbol mdrv:C
- C12: renamed from C10; value 10uF/50V -> 10uF/25V; MPN TDK C2012X5R1H106K125AC (X5R 2012) ※50V/10uF は 1608 の量産品なし -> Murata GRM21BR61E106KA73L (X5R 2012)
- C14: renamed from C12; value 10uF/25V -> 4.7uF/16V; MPN Murata GRM188R61E106MA73D (X5R 1608) -> Samsung CL10A475KO8NNNC (X5R 1608)
- C16: renamed from R13; value 1k -> 10nF/50V; footprint Resistor_SMD:R_0402_1005Metric -> Capacitor_SMD:C_0402_1005Metric; symbol mdrv:R -> mdrv:C; MPN (none) -> Murata GRM155R71H103KA88D (X7R 1005)
- C17: renamed from C15; value 0.1uF/50V -> 1nF C0G; MPN Murata GRM155R71H104KE14D (X7R 1005) -> Murata GRM1555C1H102JA01D (C0G 1005)
- C18: renamed from C16; value 10nF/50V -> 0.1uF/50V; MPN Murata GRM155R71H103KA88D (X7R 1005) -> Murata GRM155R71H104KE14D (X7R 1005)
- C19: renamed from R15; value 1k 1% -> 2.2nF C0G; footprint Resistor_SMD:R_0402_1005Metric -> Capacitor_SMD:C_0402_1005Metric; symbol mdrv:R -> mdrv:C; MPN (none) -> Murata GRM1555C1H222JA01D (C0G 1005)
- C20: renamed from R17; value 100R 1% -> 2.2nF C0G; footprint Resistor_SMD:R_0402_1005Metric -> Capacitor_SMD:C_0402_1005Metric; symbol mdrv:R -> mdrv:C; MPN (none) -> Murata GRM1555C1H222JA01D (C0G 1005)
- C21: renamed from C19; value 2.2nF C0G -> 2.2uF/25V; footprint Capacitor_SMD:C_0402_1005Metric -> Capacitor_SMD:C_0603_1608Metric; MPN Murata GRM1555C1H222JA01D (C0G 1005) -> Murata GRM188R61E225KA12D (X5R 1608)
- C22: renamed from R18; value 100R 1% -> 2.2uF/25V; footprint Resistor_SMD:R_0402_1005Metric -> Capacitor_SMD:C_0603_1608Metric; symbol mdrv:R -> mdrv:C; MPN (none) -> Murata GRM188R61E225KA12D (X5R 1608)
- C23: renamed from R19; value 100R 1% -> 2.2uF/25V; footprint Resistor_SMD:R_0402_1005Metric -> Capacitor_SMD:C_0603_1608Metric; symbol mdrv:R -> mdrv:C; MPN (none) -> Murata GRM188R61E225KA12D (X5R 1608)
- C24: renamed from C20; value 2.2nF C0G -> 2.2uF/25V; footprint Capacitor_SMD:C_0402_1005Metric -> Capacitor_SMD:C_0603_1608Metric; MPN Murata GRM1555C1H222JA01D (C0G 1005) -> Murata GRM188R61E225KA12D (X5R 1608)
- R13: renamed from C14; value 4.7uF/10V -> 1k; footprint Capacitor_SMD:C_0402_1005Metric -> Resistor_SMD:R_0402_1005Metric; symbol mdrv:C -> mdrv:R; MPN Murata GRM155R61A475MEAAD (X5R 1005) -> (none)
- R14: renamed from R11; value 110k 1% -> 12k 1%; MPN 24V 系は 180k 1% -> (none)
- R15: renamed from R12; value 10k 1% -> 1k 1%
- R16: renamed from C17; value 1nF C0G -> 100R 1%; footprint Capacitor_SMD:C_0402_1005Metric -> Resistor_SMD:R_0402_1005Metric; symbol mdrv:C -> mdrv:R; MPN Murata GRM1555C1H102JA01D (C0G 1005) -> (none)
- R17: renamed from R14; value 12k 1% -> 100R 1%
- R18: renamed from C18; value 0.1uF/50V -> 100R 1%; footprint Capacitor_SMD:C_0402_1005Metric -> Resistor_SMD:R_0402_1005Metric; symbol mdrv:C -> mdrv:R; MPN Murata GRM155R71H104KE14D (X7R 1005) -> (none)
- renumbered C11 to C13, C13 to C15, R16 to R19
Connections:
- net VBUS is gone; now on net +3V3: R14.1
- net +3V3: now also C14.1, C15.1; no longer C17.1, R13.1, R17.1
- net GND: now also C16.2, C10.2, C11.2; no longer C19.2, R13.2, R16.2, R18.2
- net IA_N: now also C19.2, R17.2; no longer C20.2, C21.2
- net IA_P: now also C19.1, R16.2; no longer C21.1, R19.2
- net IBUS_F: now also C17.1, R13.2; no longer C16.2, R16.1
- net IB_N: now also C20.2, R19.2; no longer C23.2, C24.2
- net IB_P: now also C20.1, R18.2; no longer C22.2, C24.1
- net ISA_SEL: now also R16.1; no longer R19.1
- net ISB_SEL: now also R18.1; no longer C22.1
- net ISH: now also R13.1, R17.1, R19.1; no longer C16.1, C20.1, C23.1
- net OCP_REF: now also C18.1, R14.2, R15.1; no longer C19.1, R17.2, R18.1
- net SW0: now also C21.2
- net SW1: now also C22.2
- net SW2: now also C23.2
- net SW3: now also C24.2
- net VB0: now also C21.1
- net VB1: now also C22.1
- net VB2: now also C23.1
- net VB3: now also C24.1
- net VBUS_SNS: now also C16.1; no longer C18.1, R14.2, R15.1
- net VDD8: now also C12.1, C13.1; no longer C14.1, C15.1
- net VHV: now also C10.1, C11.1; no longer C12.1, C13.1
Other:
- note added: "2.2uF 1608 (DC バイアス後 ≈1.3uF): Qg 41nC で降下 32mV, Qg ≈150nC でも ≈0.12V。"
- note added: "OPA3 出力 → ADC_IN9, OPA4 出力 → ADC_IN10 (チップ内部接続)。ゲイン 4/8/16/55。"
- note added: "PB3: バス電流 (10mΩ: 1A = 10mV) + CMP3_P3。PB2: 閾値 254mV (25.4A) = CMP3_N3。"
- note added: "VBUS_SNS (PB4 = ADC17 + OVP リセット) の分圧抵抗は子基板側 (電圧系ごとに定数が違う)。C16 は MCU 直近の平滑。"
- note added: "VHV 5〜28V (≥10uF, 1206/50V)。VDD8 5/8/9/10V (≥10uF, 2012/25V)。VDD33 4.7uF (1608/16V)。"
- note added: "バス電流フィルタ / 過電流比較の閾値"
- note added: "ブートストラップ容量 (VBx-VSx, MCU ピン直近)"
- note added: "電源デカップリング (ピン直近)"
- note removed: "2.2uF (1608, DC バイアス後 ≈1.3uF): Qg 41nC (A) で降下 32mV, Qg ≈150nC (B) でも ≈0.12V。"
- note removed: "3 相センシング PA5/PA6/PA7 = CMP3 N0/N1/N2 (仮想中性点 + TIM2 キャプチャ) = TIM2 CH1/2/3 (ホール XOR)"
- note removed: "CMP2: P=OPA3 出力, N=内蔵 DAC (0.1〜3.1V/0.2V) → TIM1 BKIN。"
- note removed: "I2C: PA14/PA15 (リマップ2)。UART: PC1/PC2 (リマップ1)。RST: PC0。SDI 1 線: PA3。水晶: PB5/PB6"
- note removed: "ISH / ISA_SEL / ISB_SEL は子基板のシャントから J10 経由で来る (ケルビン配線)。"
- note removed: "J6 引き出し: PC4 (USER/BOOT + 状態 LED), PC5 (HV I/O), TACH_IN, nFAULT (PA13 = TIM1_BKIN_1)"
- note removed: "OPA3 出力 → ADC_IN9, OPA4 出力 → ADC_IN10 (チップ内部接続)。電流チャネル選択 JP5/JP7 は子基板。"
- note removed: "PB3: バス電流 ADC_IN1 (10mΩ: 1A = 10mV) + CMP3_P3。PB2: 閾値 254mV (25.4A) = CMP3_N3 / ADC_IN0。"
- note removed: "PB4: VBUS/12 → ADC_IN17 + OVP リセット (1.5V → 18.0V)。24V 系は R11=180k (VBUS/19, 28.5V)。"
- note removed: "PWM: HB0〜HB2 = TIM1 (相補+ブレーキ)。HB2/HB3 を TIM2 リマップ2 (PB12〜PB15) で駆動すれば 4 レッグ全て相補"
- note removed: "QII1: PA12 → OPA1 (AV20/40) → CMP1 → TIM3 CH1 キャプチャ (JP8: タコ/VR 入力 or バス電流リップル)"
- note removed: "USB: CC1/CC2 = PA0/PA1 (PD0 シンク), D+/D- = PB0/PB1, USB VBUS 監視 = PA2, PD 給電許可 = PC3"
- note removed: "VBUS 監視・過電圧リセット / バス電流 / 過電流比較"
- note removed: "VHV 5〜28V (≥10uF)。VDD8 は FW で 5/8/9/10V 選択 (≥10uF)。VDD33 は 1〜10uF (DS 1.4.3)。"
- note removed: "ゲイン 4/8/16/55, バイアス 1.6V (10mΩ: G55=±2.9A, G16=±10A, G8=±20A)。"
- note removed: "ピン割当の要点 (QFN48 = CH32M030C8U7)"
- note removed: "ブートストラップダイオード内蔵 (平均 7mA / ピーク 70mA まで)。DS 推奨 1〜10uF。"
- note removed: "ブートストラップ容量 (VBx-VSx, MCU ピン直近 = 主基板)"
- note removed: "保護: CMP3 (PB3 vs PB2) または CMP2 (OPA3 出力 vs 内蔵 DAC) → TIM1 BKIN。PB4 OVP リセット"
- note removed: "電流: IA = OPA3 (子基板 JP7: HB0 / バス) → ADC9, IB = OPA4 (子基板 JP5: HB1 / HB2) → ADC10, IBUS = PB3"
- note removed: "電源デカップリング (ピン直近, DS 図3-1-1)"
- title: mPBCH32M030DS0  CH32M030 Universal Motor Driver - Main board -> mPBCH32M030DS0  CH32M030 motor-driver MCU module (DIP-42)
- moved on the sheet: C12, C13, C14, C15, C17, C18, C21, C24, R14, R15, R17, R19
