File: hardware/power.kicad_sch (KiCad schematic)
At the start: 29 parts, among them J1 PWR_IN, Q10 TPN1R603PL, Q9 TPN2R304PL, U2 78L05, U4 LM74700-Q1, U5 LM74700-Q1

Commit message: Rev 0.4: DIP-42 MCU module + power boards A/B/C (KiCad 8)
- MCU module: 20.32 x 53.34mm (8 x 21 grid), DIP-42 (0.6in rows), fits
  an 82 x 52mm breadboard. Headers can be fitted from either side;
  signal names on bottom silk. All LEDs (power, status, 8 gate LEDs) on
  the module top.
- Power boards take the module in two 1x21 sockets (left/right
  symmetric mating). FETs/shunts on the heatsink side, no LEDs.
  Voltage-dependent parts (TVS, OVP divider, bulk caps, BEMF divider)
  moved to the power boards. Breakout board D removed.
  A/C: 20.32 x 71.94mm, B (TO-263 x8): 40.64 x 66.94mm.
- Capacitors re-selected for realistic size vs voltage/capacitance
  (4.7uF 1608, 10uF/25V 2012, 10uF/50V 1206, 4.7nF/100V 1608, low
  profile electrolytics).
- Schematics and boards generated in KiCad 8 format; netlists verified
  with KiCad 8.0.9.
- Layout pipeline: Freerouting bridge (parallel), second pass, early
  repair before pours, island-aware maze repair, DRC via kicad-cli.
- DRC: power boards A/B/C have 0 unconnected / 0 electrical errors.
  The MCU module still has unrouted connections (work in progress).

Co-Authored-By: Claude Opus 5.5 <noreply@anthropic.com>
Claude-Session: https://claude.ai/code/session_01LENFjjhDfYjJZV1NWhB9uV
Parts:
- removed C1: 10uF/50V, Capacitor_SMD:C_0805_2012Metric, symbol mdrv:C
- removed C3: 1uF/50V, Capacitor_SMD:C_0603_1608Metric, symbol mdrv:C
- removed C4: 1uF/25V, Capacitor_SMD:C_0402_1005Metric, symbol mdrv:C
- removed C5, C6: 0.1uF/50V, Capacitor_SMD:C_0402_1005Metric, symbol mdrv:C
- removed D1: SMBJ16A, Diode_SMD:D_SMB, symbol mdrv:D_TVS
- removed D9: SMAJ20A, Diode_SMD:D_SMA, symbol mdrv:D_TVS
- removed F1: 10A, mPB:Fuse_Littelfuse_NANO2_2410, symbol mdrv:FUSE
- removed F3: 5A, Fuse:Fuse_1812_4532Metric, symbol mdrv:FUSE
- removed J1: PWR_IN, Connector_PinHeader_2.54mm:PinHeader_2x04_P2.54mm_Vertical, symbol mdrv:CONN2x4
- removed Q10: TPN1R603PL, Package_SO:Vishay_PowerPAK_1212-8_Single, symbol mdrv:NMOS
- removed R3: 2.2k, Resistor_SMD:R_0402_1005Metric, symbol mdrv:R
- removed R6: 100k, Resistor_SMD:R_0402_1005Metric, symbol mdrv:R
- removed U2: 78L05, Package_TO_SOT_SMD:SOT-89-3, symbol mdrv:REG3
- removed U4, U5: LM74700-Q1, Package_TO_SOT_SMD:SOT-23-6, symbol mdrv:LM74700
- D2, D7, D8: MPN (none) -> 1608 チップ LED
- R3: renamed from Q9; value TPN2R304PL -> 2.2k; footprint Package_SO:Vishay_PowerPAK_1212-8_Single -> Resistor_SMD:R_0402_1005Metric; symbol mdrv:NMOS -> mdrv:R; MPN Toshiba TPN2R304PL,L1Q (40V 2.3mΩ, J1 側 理想ダイオード) -> (none)
Connections:
- net USB_VBUS_P is gone; now on net USB_VBUS: R7.1
- net +5V: now also R3.1
- net VBUS: no longer R3.5 (D)
- net LED_D7_A: now reaches D7.2 (A), R4.2
- net LED_D2_A: now reaches D2.2 (A)
- net LED_D2_A: now also R3.2
- net VHV_IN: now reaches D5.1 (K), D6.1 (K), R10.1
- net LED_D8_A: now reaches D8.2 (A), R5.2
- removed net Q9_G: R3.4 (G)
- removed net VIN_F: R3.1 (S), R3.2 (S), R3.3 (S)
Other:
- note added: "D7: モータ電源 VBUS D2: +5V (子基板の 78L05) D8: VDD33 (1.5k で約 0.9mA, VDD33 負荷 ≤20mA)"
- note added: "MCU 電源 VHV (VBUS ピン / USB 5V のダイオード OR + 27V クランプ)"
- note added: "R10 47Ω + D4 27V: 24V 系のサージで VHV が 30V を超えないようにする。"
- note added: "USB VBUS 監視 (PA2)"
- note added: "USB_VBUS / 13 → PA2 (20V → 1.54V)。PD 契約後の電圧確認に使う。"
- note added: "VBUS ピン (子基板のモータ電源) か USB 5V のどちらかで MCU が動く。ブレッドボード単体は USB 給電のみで可。"
- note added: "電源表示 LED (モジュール上面: 子基板を付けても見える)"
- note removed: "12V 系: D1=SMBJ16A, R11=110k (OVP 18V)。24V 系 (子基板 B): D1=SMBJ24A, R11=180k (OVP 28.5V)。"
- note removed: "5V 補助電源 (ホールセンサ用) / 電源表示 LED"
- note removed: "CH32M030 の VS 絶対最大 30V / VHV 動作 5〜28V → 24V 系は安定化電源専用 (回生・サージで 28V を超えないこと)。"
- note removed: "D7: モータ電源 (VBUS, 12V で 0.6mA / 24V で 1.5mA) D2: +5V D8: MCU 電源 (VDD33)"
- note removed: "J1 と USB-PD (下) は理想ダイオード OR。バルク容量は子基板の MOSFET 近傍に置く (C1 は局所バイパス)。"
- note removed: "J1 はピンヘッダ 4 ピン並列 (約 10A)。それ以上は J1 のランドへ線材を直接はんだ付けする。"
- note removed: "MCU 電源 VHV (VBUS / USB 5V のダイオード OR + 27V クランプ)"
- note removed: "PB4 の OVP リセットで MCU がリセットされると EN も Low → USB 給電も自動遮断。"
- note removed: "PD_PWR_EN (PC3) = Low/リセット中は OFF (R6)。FW は PS_RDY 受信 + USB_VBUS_SNS (PA2) で電圧確認後に ON。"
- note removed: "R10 47Ω + D4 27V: 24V 系のサージで VHV が 30V を超えないようにする (MCU 消費 ≤35mA で降下 ≤1.7V)。"
- note removed: "U4+Q9: 逆接続 (最大 -65V) と VBUS→J1 への逆流を阻止する理想ダイオード。Q9 は 40V 品 (24V 系と共通)。"
- note removed: "USB のみ給電では VHV < 5V となり PA0〜PA3 の出力 High が VDD33-1.7V に下がる (DS 注5)。"
- note removed: "USB のみ給電時 VHV ≈ 4.4V (≥ 4.0V で MCU 動作)。ゲート駆動は VBUS ≥ 8V を FW で確認してから許可。"
- note removed: "USB-PD 給電パス (PD 契約後に MCU が許可, 最大 15V / 5A)"
- note removed: "USB_VBUS_SNS = USB VBUS / 13 (20V → 1.54V)。"
- note removed: "VBUS の突入: 子基板のバルク容量を PD 電源で充電するため FW は EN ON 後に電流を段階的に上げる。"
- note removed: "VDD33 の負荷上限は 20mA (DS 表3-4) → D8 は 1.5k で約 0.9mA に抑える。"
- note removed: "電源入力 (J1 2x4 ピン) / 理想ダイオード (逆接・逆流防止) / サージ保護"
- title: mPBCH32M030DS0  CH32M030 Universal Motor Driver - Main board -> mPBCH32M030DS0  CH32M030 motor-driver MCU module (DIP-42)
