File: hardware/mPBCH32M030DS0.kicad_sch (KiCad schematic)
At the start: 0 parts

Commit message: Rev 0.3: パワー段を子基板化 (A/B/C/D) し 2 層基板レイアウトを作成
構成:
- 主基板 (60x42mm, 2 層): 右 = CH32M030 / USB-C / GPIO・I2C・UART・SDI・HALL,
  左上 = 電源 (J1 → F1 → 理想ダイオード, USB-PD 経路), 左下 = 基板間コネクタ J9/J10 (裏面)
- 子基板と裏面同士を背中合わせに重ねる (基板間 約5mm, 裏面部品は高さ 2mm 以下)。
  RESET / USER・BOOT / センシング選択は主基板 TOP、電流チャネル選択 JP5/JP7 は子基板 TOP
- 子基板 A: TPN1R603PL (既存回路) / B: TKR74F04PB (24V 系, 66x66mm) /
  C: MTN2306AN3 (廉価版) / D: MOSFET なし (全信号をピンヘッダへ引き出し)
- 基板間ピンは同じ番号同士が嵌合 (ソケットを 270° 回転して裏面実装, 座標で全 32 ピンを検証)
- コネクタは USB-C 以外すべて 2.54mm ピンヘッダ。コンデンサは 1005/1608 基本
  (入手性を確認した量産品番。50V/10uF のみ 2012)
- 24V 対応: Q9 を 40V 品 (TPN2R304PL), VHV に 47Ω + 27V ツェナー, D1/R11 の 24V 用定数を注記,
  FW は make POWER_STAGE=B で VBUS 分圧比を切替
- F1 を NANO2 10A (SMD), スイッチを B3U-1000P に小型化

基板生成 (hardware/gen_pcb.py + pcblib.py):
- 配置 → Freerouting 1.9 自動配線 → 大電流ネットのベタ化 → GND ベタ・スティッチング
  → 残り接続の補修 (格子 A*, DRC が増えない経路のみ採用) → DRC
- 5 基板とも未接続 0・電気的 DRC エラー 0 (警告はシルクの重なりのみ)
- 製造データ hardware/fab/*.zip (ガーバー, ドリル, 両面の部品座標)

回路図: 主基板 82/82, 子基板 A/B/C 41/41, D 21/21 ネット一致。FW は A/B とも警告 0 でビルド。

Co-Authored-By: Claude Opus 5.5 <noreply@anthropic.com>
Claude-Session: https://claude.ai/code/session_01LENFjjhDfYjJZV1NWhB9uV
Other:
- removed sheet パワー段 (4 ハーフブリッジ) / ゲート確認 LED / シャント / モータ出力
- added sheet 基板間コネクタ (子基板) / 3 相センシング選択 (b2b.kicad_sch)
- note added: "mPBCH32M030DS0 Rev 0.3 主基板 — CH32M030C8U7 (QFN48) ユニバーサル・モータードライバ (3相 ・ DC x2 ・ ステッピング)"
- note added: "・2 層基板 60 x 42mm。部品面 (TOP): 右 = MCU / USB-C / GPIO・I2C・UART・SDI・HALL, 左上 = 電源, 左下 = 基板間コネクタ"
- note added: "・3 相センシング PA5/PA6/PA7 (CMP3 + 仮想中性点 + TIM2) / ホール XOR, QII1 タコ入力, NTC (子基板の MOSFET 近傍)"
- note added: "・PWM: HB0〜HB2 = TIM1, HB2/HB3 = TIM2 リマップ2。電流: OPA3/OPA4 → ADC, CMP3 or CMP2(+DAC) → TIM1 ブレーキ"
- note added: "・コネクタはすべて 2.54mm ピンヘッダ (USB-C を除く)。操作系 (RESET, USER/BOOT, センシング選択 JP2-4/JP8) は TOP 面"
- note added: "・パワー段 (MOSFET x8, シャント, ゲート確認 LED, 相電圧分圧, NTC, バルク容量) は子基板へ分離し, 裏面同士を"
- note added: "・電源: J1 (2x4 ピン, 8〜16V / 24V 系は注記の部品に変更) と USB-C PD (9/12/15V) を理想ダイオード OR"
- note added: "向かい合わせて J9 (電源 2x5) / J10 (信号 2x11) で接続する (基板間 約5mm, 裏面部品は高さ 2mm 以下)。"
- note added: "子基板 A: TPN1R603PL (既存回路, 8〜16V) B: TKR74F04PB (24V 系) C: MTN2306AN3 (廉価, ≤3A) D: MOSFET なし (ピン出し)"
- note added: "詳細は README.md, docs/design.md, docs/stacking.md, docs/advanced_features.md を参照。"
- note removed: "3相 FOC : U=OUT0 V=OUT1 W=OUT2 JP5=1-2 JP7=1-2 保護 CMP3(バス)+CMP2(IA)"
- note removed: "3相 センサレス 6 ステップ : 同上 JP7=2-3 (バス) CMP3 = BEMF, 保護 CMP2(バス)"
- note removed: "DC x2 / ステッピング : A+=OUT0 A-=OUT1 B+=OUT2 B-=OUT3 JP5=2-3 JP7=1-2"
- note removed: "mPBCH32M030DS0 Rev 0.2 — CH32M030C8U7 (QFN48) ユニバーサル・モータードライバ (3相 ・ DC x2 ・ ステッピング)"
- note removed: "・3 相センシング PA5/PA6/PA7: CMP3 + 内部仮想中性点 + TIM2 キャプチャ (センサレス) / TIM2 ホール XOR / ISOURCE 自己診断"
- note removed: "・PWM: HB0〜HB2 = TIM1, HB2/HB3 = TIM2 リマップ2 (4 レッグ相補)。ゲート確認 LED x8, 電源 LED x3"
- note removed: "・QII1 (OPA1+CMP1 → TIM3): タコ・VR センサ入力, ブラシ DC の電流リップル計数 (JP8)"
- note removed: "・USB-C: USB2.0 FS (ブートローダ書き込み) + PD シンク。RESET, USER/BOOT(+状態 LED), 8MHz 水晶"
- note removed: "・電流: IA = OPA3 (JP7: HB0/バス), IB = OPA4 (JP5: HB1/HB2), IBUS = PB3 直接。CMP3 or CMP2(+DAC) → TIM1 ブレーキ"
- note removed: "・電源: J1 8〜16V と USB-C PD (9/12/15V, ≤5A) を理想ダイオード OR (LM74700 + TPN1R603PL x2)。PD は契約後に MCU が許可"
- note removed: "詳細設計・部品選定・内蔵機能の活用検討は README.md, docs/design.md, docs/advanced_features.md を参照。"
- note removed: "駆動モード対応表 (J2 の結線)"
- title: mPBCH32M030DS0  CH32M030 Universal Motor Driver -> mPBCH32M030DS0  CH32M030 Universal Motor Driver - Main board
Changed lines of the file:
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@@
 (kicad_sch (version 20230121) (generator eeschema)
 (paper "A3")
-(title_block (title "mPBCH32M030DS0  CH32M030 Universal Motor Driver") (date "2026-09-24") (rev "0.2") (company "ghostinkoma") (comment 1 "トップシート / 仕様概要") (comment 2 "個人利用可 (クレジット表示必須) / 商用利用は要連絡 / 無保証  -  LICENSE 参照"))
-(text "mPBCH32M030DS0 Rev 0.2 — CH32M030C8U7 (QFN48) ユニバーサル・モータードライバ (3相 ・ DC x2 ・ ステッピング)" (at 20 30 0) (effects (font (size 2 2)) (justify left bottom)))
+(title_block (title "mPBCH32M030DS0  CH32M030 Universal Motor Driver - Main board") (date "2026-09-25") (rev "0.3") (company "ghostinkoma") (comment 1 "トップシート / 仕様概要") (comment 2 "個人利用可 (クレジット表示必須) / 商用利用は要連絡 / 無保証  -  LICENSE 参照"))
+(text "mPBCH32M030DS0 Rev 0.3 主基板 — CH32M030C8U7 (QFN48) ユニバーサル・モータードライバ (3相 ・ DC x2 ・ ステッピング)" (at 20 30 0) (effects (font (size 2 2)) (justify left bottom)))
 (text "" (at 20 37 0) (effects (font (size 2 2)) (justify left bottom)))
-(text "・電源: J1 8〜16V と USB-C PD (9/12/15V, ≤5A) を理想ダイオード OR (LM74700 + TPN1R603PL x2)。PD は契約後に MCU が許可" (at 20 44 0) (effects (font (size 2 2)) (justify left bottom)))
-(text "・PWM: HB0〜HB2 = TIM1, HB2/HB3 = TIM2 リマップ2 (4 レッグ相補)。ゲート確認 LED x8, 電源 LED x3" (at 20 51 0) (effects (font (size 2 2)) (justify left bottom)))
-(text "・電流: IA = OPA3 (JP7: HB0/バス), IB = OPA4 (JP5: HB1/HB2), IBUS = PB3 直接。CMP3 or CMP2(+DAC) → TIM1 ブレーキ" (at 20 58 0) (effects (font (size 2 2)) (justify left bottom)))
-(text "・3 相センシング PA5/PA6/PA7: CMP3 + 内部仮想中性点 + TIM2 キャプチャ (センサレス) / TIM2 ホール XOR / ISOURCE 自己診断" (at 20 65 0) (effects (font (size 2 2)) (justify left bottom)))
-(text "・QII1 (OPA1+CMP1 → TIM3): タコ・VR センサ入力, ブラシ DC の電流リップル計数 (JP8)" (at 20 72 0) (effects (font (size 2 2)) (justify left bottom)))
-(text "・USB-C: USB2.0 FS (ブートローダ書き込み) + PD シンク。RESET, USER/BOOT(+状態 LED), 8MHz 水晶" (at 20 79 0) (effects (font (size 2 2)) (justify left bottom)))
-(text "" (at 20 86 0) (effects (font (size 2 2)) (justify left bottom)))
-(text "駆動モード対応表 (J2 の結線)" (at 20 93 0) (effects (font (size 2 2)) (justify left bottom)))
-(text "  3相 FOC       : U=OUT0 V=OUT1 W=OUT2   JP5=1-2 JP7=1-2  保護 CMP3(バス)+CMP2(IA)" (at 20 100 0) (effects (font (size 2 2)) (justify left bottom)))
-(text "  3相 センサレス 6 ステップ : 同上        JP7=2-3 (バス)  CMP3 = BEMF, 保護 CMP2(バス)" (at 20 107 0) (effects (font (size 2 2)) (justify left bottom)))
-(text "  DC x2 / ステッピング : A+=OUT0 A-=OUT1 B+=OUT2 B-=OUT3  JP5=2-3 JP7=1-2" (at 20 114 0) (effects (font (size 2 2)) (justify left bottom)))
-(text "" (at 20 121 0) (effects (font (size 2 2)) (justify left bottom)))
-(text "詳細設計・部品選定・内蔵機能の活用検討は README.md, docs/design.md, docs/advanced_features.md を参照。" (at 20 128 0) (effects (font (size 2 2)) (justify left bottom)))
-(sheet (at 20 160) (size 70 30) (fields_autoplaced) (stroke (width 0.1524) (type solid)) (fill (color 0 0 0 0.0000))
-(property "Sheetname" "電源入力・保護・補助電源・電源表示" (at 20 159.3 0) (effects (font (size 1.5 1.5)) (justify left bottom)))
-(property "Sheetfile" "power.kicad_sch" (at 20 190.6 0) (effects (font (size 1.27 1.27)) (justify left top)))
-(instances (project "mPBCH32M030DS0" (path "/cb038f79-02b6-58e4-b0e9-4ee93e4d05b7" (page "2"))))
+(text "・2 層基板 60 x 42mm。部品面 (TOP): 右 = MCU / USB-C / GPIO・I2C・UART・SDI・HALL, 左上 = 電源, 左下 = 基板間コネクタ" (at 20 44 0) (effects (font (size 2 2)) (justify left bottom)))
+(text "・パワー段 (MOSFET x8, シャント, ゲート確認 LED, 相電圧分圧, NTC, バルク容量) は子基板へ分離し, 裏面同士を" (at 20 51 0) (effects (font (size 2 2)) (justify left bottom)))
+(text "  向かい合わせて J9 (電源 2x5) / J10 (信号 2x11) で接続する (基板間 約5mm, 裏面部品は高さ 2mm 以下)。" (at 20 58 0) (effects (font (size 2 2)) (justify left bottom)))
+(text "   子基板 A: TPN1R603PL (既存回路, 8〜16V)   B: TKR74F04PB (24V 系)   C: MTN2306AN3 (廉価, ≤3A)   D: MOSFET なし (ピン出し)" (at 20 65 0) (effects (font (size 2 2)) (justify left bottom)))
+(text "・コネクタはすべて 2.54mm ピンヘッダ (USB-C を除く)。操作系 (RESET, USER/BOOT, センシング選択 JP2-4/JP8) は TOP 面" (at 20 72 0) (effects (font (size 2 2)) (justify left bottom)))
+(text "・電源: J1 (2x4 ピン, 8〜16V / 24V 系は注記の部品に変更) と USB-C PD (9/12/15V) を理想ダイオード OR" (at 20 79 0) (effects (font (size 2 2)) (justify left bottom)))
+(text "・PWM: HB0〜HB2 = TIM1, HB2/HB3 = TIM2 リマップ2。電流: OPA3/OPA4 → ADC, CMP3 or CMP2(+DAC) → TIM1 ブレーキ" (at 20 86 0) (effects (font (size 2 2)) (justify left bottom)))
+(text "・3 相センシング PA5/PA6/PA7 (CMP3 + 仮想中性点 + TIM2) / ホール XOR, QII1 タコ入力, NTC (子基板の MOSFET 近傍)" (at 20 93 0) (effects (font (size 2 2)) (justify left bottom)))
+(text "" (at 20 100 0) (effects (font (size 2 2)) (justify left bottom)))
+(text "詳細は README.md, docs/design.md, docs/stacking.md, docs/advanced_features.md を参照。" (at 20 107 0) (effects (font (size 2 2)) (justify left bottom)))
+(sheet (at 20 200) (size 70 30) (fields_autoplaced) (stroke (width 0.1524) (type solid)) (fill (color 0 0 0 0.0000))
+(property "Sheetname" "電源入力・保護・補助電源・電源表示" (at 20 199.3 0) (effects (font (size 1.5 1.5)) (justify left bottom)))
+(property "Sheetfile" "power.kicad_sch" (at 20 230.6 0) (effects (font (size 1.27 1.27)) (justify left top)))
+(instances (project "mPBCH32M030DS0" (path "/87b4cdf7-ae48-57cd-a772-8ad5802448bf" (page "2"))))
 )
-(sheet (at 98 160) (size 70 30) (fields_autoplaced) (stroke (width 0.1524) (type solid)) (fill (color 0 0 0 0.0000))
-(property "Sheetname" "USB Type-C / 水晶発振子 / リセット" (at 98 159.3 0) (effects (font (size 1.5 1.5)) (justify left bottom)))
-(property "Sheetfile" "usb.kicad_sch" (at 98 190.6 0) (effects (font (size 1.27 1.27)) (justify left top)))
-(instances (project "mPBCH32M030DS0" (path "/cb038f79-02b6-58e4-b0e9-4ee93e4d05b7" (page "3"))))
+(sheet (at 98 200) (size 70 30) (fields_autoplaced) (stroke (width 0.1524) (type solid)) (fill (color 0 0 0 0.0000))
+(property "Sheetname" "USB Type-C / 水晶発振子 / リセット" (at 98 199.3 0) (effects (font (size 1.5 1.5)) (justify left bottom)))
+(property "Sheetfile" "usb.kicad_sch" (at 98 230.6 0) (effects (font (size 1.27 1.27)) (justify left top)))
+(instances (project "mPBCH32M030DS0" (path "/87b4cdf7-ae48-57cd-a772-8ad5802448bf" (page "3"))))
 )
-(sheet (at 176 160) (size 70 30) (fields_autoplaced) (stroke (width 0.1524) (type solid)) (fill (color 0 0 0 0.0000))
-(property "Sheetname" "CH32M030C8U7 (QFN48) / ゲートドライバ周辺" (at 176 159.3 0) (effects (font (size 1.5 1.5)) (justify left bottom)))
-(property "Sheetfile" "mcu.kicad_sch" (at 176 190.6 0) (effects (font (size 1.27 1.27)) (justify left top)))
-(instances (project "mPBCH32M030DS0" (path "/cb038f79-02b6-58e4-b0e9-4ee93e4d05b7" (page "4"))))
+(sheet (at 176 200) (size 70 30) (fields_autoplaced) (stroke (width 0.1524) (type solid)) (fill (color 0 0 0 0.0000))
+(property "Sheetname" "CH32M030C8U7 (QFN48) / ゲートドライバ周辺" (at 176 199.3 0) (effects (font (size 1.5 1.5)) (justify left bottom)))
+(property "Sheetfile" "mcu.kicad_sch" (at 176 230.6 0) (effects (font (size 1.27 1.27)) (justify left top)))
+(instances (project "mPBCH32M030DS0" (path "/87b4cdf7-ae48-57cd-a772-8ad5802448bf" (page "4"))))
 )
-(sheet (at 254 160) (size 70 30) (fields_autoplaced) (stroke (width 0.1524) (type solid)) (fill (color 0 0 0 0.0000))
-(property "Sheetname" "パワー段 (4 ハーフブリッジ) / ゲート確認 LED / シャント / モータ出力" (at 254 159.3 0) (effects (font (size 1.5 1.5)) (justify left bottom)))
-(property "Sheetfile" "bridge.kicad_sch" (at 254 190.6 0) (effects (font (size 1.27 1.27)) (justify left top)))
-(instances (project "mPBCH32M030DS0" (path "/cb038f79-02b6-58e4-b0e9-4ee93e4d05b7" (page "5"))))
+(sheet (at 254 200) (size 70 30) (fields_autoplaced) (stroke (width 0.1524) (type solid)) (fill (color 0 0 0 0.0000))
+(property "Sheetname" "基板間コネクタ (子基板) / 3 相センシング選択" (at 254 199.3 0) (effects (font (size 1.5 1.5)) (justify left bottom)))
+(property "Sheetfile" "b2b.kicad_sch" (at 254 230.6 0) (effects (font (size 1.27 1.27)) (justify left top)))
+(instances (project "mPBCH32M030DS0" (path "/87b4cdf7-ae48-57cd-a772-8ad5802448bf" (page "5"))))
 )
-(sheet (at 332 160) (size 70 30) (fields_autoplaced) (stroke (width 0.1524) (type solid)) (fill (color 0 0 0 0.0000))
-(property "Sheetname" "インターフェース (ホール / 通信 / GPIO 引き出し / UI)" (at 332 159.3 0) (effects (font (size 1.5 1.5)) (justify left bottom)))
-(property "Sheetfile" "io.kicad_sch" (at 332 190.6 0) (effects (font (size 1.27 1.27)) (justify left top)))
-(instances (project "mPBCH32M030DS0" (path "/cb038f79-02b6-58e4-b0e9-4ee93e4d05b7" (page "6"))))
+(sheet (at 332 200) (size 70 30) (fields_autoplaced) (stroke (width 0.1524) (type solid)) (fill (color 0 0 0 0.0000))
+(property "Sheetname" "インターフェース (ホール / 通信 / GPIO 引き出し / UI)" (at 332 199.3 0) (effects (font (size 1.5 1.5)) (justify left bottom)))
+(property "Sheetfile" "io.kicad_sch" (at 332 230.6 0) (effects (font (size 1.27 1.27)) (justify left top)))
+(instances (project "mPBCH32M030DS0" (path "/87b4cdf7-ae48-57cd-a772-8ad5802448bf" (page "6"))))
 )
 (sheet_instances (path "/" (page "1")))

Commit message: Rev 0.4: DIP-42 MCU module + power boards A/B/C (KiCad 8)
- MCU module: 20.32 x 53.34mm (8 x 21 grid), DIP-42 (0.6in rows), fits
  an 82 x 52mm breadboard. Headers can be fitted from either side;
  signal names on bottom silk. All LEDs (power, status, 8 gate LEDs) on
  the module top.
- Power boards take the module in two 1x21 sockets (left/right
  symmetric mating). FETs/shunts on the heatsink side, no LEDs.
  Voltage-dependent parts (TVS, OVP divider, bulk caps, BEMF divider)
  moved to the power boards. Breakout board D removed.
  A/C: 20.32 x 71.94mm, B (TO-263 x8): 40.64 x 66.94mm.
- Capacitors re-selected for realistic size vs voltage/capacitance
  (4.7uF 1608, 10uF/25V 2012, 10uF/50V 1206, 4.7nF/100V 1608, low
  profile electrolytics).
- Schematics and boards generated in KiCad 8 format; netlists verified
  with KiCad 8.0.9.
- Layout pipeline: Freerouting bridge (parallel), second pass, early
  repair before pours, island-aware maze repair, DRC via kicad-cli.
- DRC: power boards A/B/C have 0 unconnected / 0 electrical errors.
  The MCU module still has unrouted connections (work in progress).

Co-Authored-By: Claude Opus 5.5 <noreply@anthropic.com>
Claude-Session: https://claude.ai/code/session_01LENFjjhDfYjJZV1NWhB9uV
Other:
- sheet インターフェース (ホール / 通信 / GPIO 引き出し / UI) renamed DIP 端子 J1/J2 / ゲート確認 LED / センシング選択 / I/O
- sheet 電源入力・保護・補助電源・電源表示 renamed MCU 電源 (VHV) / 電源表示 LED / USB VBUS 監視
- removed sheet 基板間コネクタ (子基板) / 3 相センシング選択
- note added: "mPBCH32M030DS0 Rev 0.4 MCU モジュール — CH32M030C8U7 (QFN48), ブレッドボード対応 DIP-42 (列間 0.6in)"
- note added: "ピンヘッダは裏から (ブレッドボード / 子基板用) でも表から (ジャンパワイヤ用) でも実装できる"
- note added: "・2 層 20.32 x 53.34mm (2.54mm 格子で 8 x 21 マス)。左右 21 ピン x 2 列, 列間 15.24mm"
- note added: "・LED はすべてモジュール上 (子基板の部品面はヒートシンク側のため): 電源 x3, 状態, ゲート確認 x8"
- note added: "・パワー段子基板 (A: TPN1R603PL / B: TKR74F04PB 24V / C: MTN2306AN3) は左右対称のピンソケットで受ける"
- note added: "・左列 J1: USB VBUS / 電源 / SDI / センサ (相電圧・ホール・電流・NTC)。右列 J2: ゲート駆動 x12 / UART / I2C / GPIO"
- note added: "・電圧に依存する部品 (TVS, VBUS 分圧, バルク容量) は子基板側。モジュールは電圧に依存しない"
- note added: "詳細は README.md, docs/stacking.md, docs/design.md を参照。"
- note removed: "mPBCH32M030DS0 Rev 0.3 主基板 — CH32M030C8U7 (QFN48) ユニバーサル・モータードライバ (3相 ・ DC x2 ・ ステッピング)"
- note removed: "・2 層基板 60 x 42mm。部品面 (TOP): 右 = MCU / USB-C / GPIO・I2C・UART・SDI・HALL, 左上 = 電源, 左下 = 基板間コネクタ"
- note removed: "・3 相センシング PA5/PA6/PA7 (CMP3 + 仮想中性点 + TIM2) / ホール XOR, QII1 タコ入力, NTC (子基板の MOSFET 近傍)"
- note removed: "・PWM: HB0〜HB2 = TIM1, HB2/HB3 = TIM2 リマップ2。電流: OPA3/OPA4 → ADC, CMP3 or CMP2(+DAC) → TIM1 ブレーキ"
- note removed: "・コネクタはすべて 2.54mm ピンヘッダ (USB-C を除く)。操作系 (RESET, USER/BOOT, センシング選択 JP2-4/JP8) は TOP 面"
- note removed: "・パワー段 (MOSFET x8, シャント, ゲート確認 LED, 相電圧分圧, NTC, バルク容量) は子基板へ分離し, 裏面同士を"
- note removed: "・電源: J1 (2x4 ピン, 8〜16V / 24V 系は注記の部品に変更) と USB-C PD (9/12/15V) を理想ダイオード OR"
- note removed: "向かい合わせて J9 (電源 2x5) / J10 (信号 2x11) で接続する (基板間 約5mm, 裏面部品は高さ 2mm 以下)。"
- note removed: "子基板 A: TPN1R603PL (既存回路, 8〜16V) B: TKR74F04PB (24V 系) C: MTN2306AN3 (廉価, ≤3A) D: MOSFET なし (ピン出し)"
- note removed: "詳細は README.md, docs/design.md, docs/stacking.md, docs/advanced_features.md を参照。"
- title: mPBCH32M030DS0  CH32M030 Universal Motor Driver - Main board -> mPBCH32M030DS0  CH32M030 motor-driver MCU module (DIP-42)
Changed lines of the file:
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@@
-(kicad_sch (version 20230121) (generator eeschema)
+(kicad_sch (version 20231120) (generator "eeschema") (generator_version "8.0")
 (paper "A3")
-(title_block (title "mPBCH32M030DS0  CH32M030 Universal Motor Driver - Main board") (date "2026-09-25") (rev "0.3") (company "ghostinkoma") (comment 1 "トップシート / 仕様概要") (comment 2 "個人利用可 (クレジット表示必須) / 商用利用は要連絡 / 無保証  -  LICENSE 参照"))
-(text "mPBCH32M030DS0 Rev 0.3 主基板 — CH32M030C8U7 (QFN48) ユニバーサル・モータードライバ (3相 ・ DC x2 ・ ステッピング)" (at 20 30 0) (effects (font (size 2 2)) (justify left bottom)))
-(text "" (at 20 37 0) (effects (font (size 2 2)) (justify left bottom)))
-(text "・2 層基板 60 x 42mm。部品面 (TOP): 右 = MCU / USB-C / GPIO・I2C・UART・SDI・HALL, 左上 = 電源, 左下 = 基板間コネクタ" (at 20 44 0) (effects (font (size 2 2)) (justify left bottom)))
-(text "・パワー段 (MOSFET x8, シャント, ゲート確認 LED, 相電圧分圧, NTC, バルク容量) は子基板へ分離し, 裏面同士を" (at 20 51 0) (effects (font (size 2 2)) (justify left bottom)))
-(text "  向かい合わせて J9 (電源 2x5) / J10 (信号 2x11) で接続する (基板間 約5mm, 裏面部品は高さ 2mm 以下)。" (at 20 58 0) (effects (font (size 2 2)) (justify left bottom)))
-(text "   子基板 A: TPN1R603PL (既存回路, 8〜16V)   B: TKR74F04PB (24V 系)   C: MTN2306AN3 (廉価, ≤3A)   D: MOSFET なし (ピン出し)" (at 20 65 0) (effects (font (size 2 2)) (justify left bottom)))
-(text "・コネクタはすべて 2.54mm ピンヘッダ (USB-C を除く)。操作系 (RESET, USER/BOOT, センシング選択 JP2-4/JP8) は TOP 面" (at 20 72 0) (effects (font (size 2 2)) (justify left bottom)))
-(text "・電源: J1 (2x4 ピン, 8〜16V / 24V 系は注記の部品に変更) と USB-C PD (9/12/15V) を理想ダイオード OR" (at 20 79 0) (effects (font (size 2 2)) (justify left bottom)))
-(text "・PWM: HB0〜HB2 = TIM1, HB2/HB3 = TIM2 リマップ2。電流: OPA3/OPA4 → ADC, CMP3 or CMP2(+DAC) → TIM1 ブレーキ" (at 20 86 0) (effects (font (size 2 2)) (justify left bottom)))
-(text "・3 相センシング PA5/PA6/PA7 (CMP3 + 仮想中性点 + TIM2) / ホール XOR, QII1 タコ入力, NTC (子基板の MOSFET 近傍)" (at 20 93 0) (effects (font (size 2 2)) (justify left bottom)))
-(text "" (at 20 100 0) (effects (font (size 2 2)) (justify left bottom)))
-(text "詳細は README.md, docs/design.md, docs/stacking.md, docs/advanced_features.md を参照。" (at 20 107 0) (effects (font (size 2 2)) (justify left bottom)))
-(sheet (at 20 200) (size 70 30) (fields_autoplaced) (stroke (width 0.1524) (type solid)) (fill (color 0 0 0 0.0000))
-(property "Sheetname" "電源入力・保護・補助電源・電源表示" (at 20 199.3 0) (effects (font (size 1.5 1.5)) (justify left bottom)))
+(title_block (title "mPBCH32M030DS0  CH32M030 motor-driver MCU module (DIP-42)") (date "2026-09-26") (rev "0.4") (company "ghostinkoma") (comment 1 "トップシート / 仕様概要") (comment 2 "個人利用可 (クレジット表示必須) / 商用利用は要連絡 / 無保証  -  LICENSE 参照"))
+(text "mPBCH32M030DS0 Rev 0.4 MCU モジュール — CH32M030C8U7 (QFN48), ブレッドボード対応 DIP-42 (列間 0.6in)" (exclude_from_sim no) (at 20 30 0) (effects (font (size 2 2)) (justify left bottom)))
+(text "" (exclude_from_sim no) (at 20 37 0) (effects (font (size 2 2)) (justify left bottom)))
+(text "・2 層 20.32 x 53.34mm (2.54mm 格子で 8 x 21 マス)。左右 21 ピン x 2 列, 列間 15.24mm" (exclude_from_sim no) (at 20 44 0) (effects (font (size 2 2)) (justify left bottom)))
+(text "  ピンヘッダは裏から (ブレッドボード / 子基板用) でも表から (ジャンパワイヤ用) でも実装できる" (exclude_from_sim no) (at 20 51 0) (effects (font (size 2 2)) (justify left bottom)))
+(text "・左列 J1: USB VBUS / 電源 / SDI / センサ (相電圧・ホール・電流・NTC)。右列 J2: ゲート駆動 x12 / UART / I2C / GPIO" (exclude_from_sim no) (at 20 58 0) (effects (font (size 2 2)) (justify left bottom)))
+(text "・LED はすべてモジュール上 (子基板の部品面はヒートシンク側のため): 電源 x3, 状態, ゲート確認 x8" (exclude_from_sim no) (at 20 65 0) (effects (font (size 2 2)) (justify left bottom)))
+(text "・パワー段子基板 (A: TPN1R603PL / B: TKR74F04PB 24V / C: MTN2306AN3) は左右対称のピンソケットで受ける" (exclude_from_sim no) (at 20 72 0) (effects (font (size 2 2)) (justify left bottom)))
+(text "・電圧に依存する部品 (TVS, VBUS 分圧, バルク容量) は子基板側。モジュールは電圧に依存しない" (exclude_from_sim no) (at 20 79 0) (effects (font (size 2 2)) (justify left bottom)))
+(text "" (exclude_from_sim no) (at 20 86 0) (effects (font (size 2 2)) (justify left bottom)))
+(text "詳細は README.md, docs/stacking.md, docs/design.md を参照。" (exclude_from_sim no) (at 20 93 0) (effects (font (size 2 2)) (justify left bottom)))
+(sheet (at 20 200) (size 70 30) (fields_autoplaced yes) (stroke (width 0.1524) (type solid)) (fill (color 0 0 0 0.0000))
+(property "Sheetname" "MCU 電源 (VHV) / 電源表示 LED / USB VBUS 監視" (at 20 199.3 0) (effects (font (size 1.5 1.5)) (justify left bottom)))
 (property "Sheetfile" "power.kicad_sch" (at 20 230.6 0) (effects (font (size 1.27 1.27)) (justify left top)))
 (instances (project "mPBCH32M030DS0" (path "/87b4cdf7-ae48-57cd-a772-8ad5802448bf" (page "2"))))
 )
-(sheet (at 98 200) (size 70 30) (fields_autoplaced) (stroke (width 0.1524) (type solid)) (fill (color 0 0 0 0.0000))
+(sheet (at 98 200) (size 70 30) (fields_autoplaced yes) (stroke (width 0.1524) (type solid)) (fill (color 0 0 0 0.0000))
 (property "Sheetname" "USB Type-C / 水晶発振子 / リセット" (at 98 199.3 0) (effects (font (size 1.5 1.5)) (justify left bottom)))
 (property "Sheetfile" "usb.kicad_sch" (at 98 230.6 0) (effects (font (size 1.27 1.27)) (justify left top)))
 (instances (project "mPBCH32M030DS0" (path "/87b4cdf7-ae48-57cd-a772-8ad5802448bf" (page "3"))))
 )
-(sheet (at 176 200) (size 70 30) (fields_autoplaced) (stroke (width 0.1524) (type solid)) (fill (color 0 0 0 0.0000))
+(sheet (at 176 200) (size 70 30) (fields_autoplaced yes) (stroke (width 0.1524) (type solid)) (fill (color 0 0 0 0.0000))
 (property "Sheetname" "CH32M030C8U7 (QFN48) / ゲートドライバ周辺" (at 176 199.3 0) (effects (font (size 1.5 1.5)) (justify left bottom)))
 (property "Sheetfile" "mcu.kicad_sch" (at 176 230.6 0) (effects (font (size 1.27 1.27)) (justify left top)))
 (instances (project "mPBCH32M030DS0" (path "/87b4cdf7-ae48-57cd-a772-8ad5802448bf" (page "4"))))
 )
-(sheet (at 254 200) (size 70 30) (fields_autoplaced) (stroke (width 0.1524) (type solid)) (fill (color 0 0 0 0.0000))
-(property "Sheetname" "基板間コネクタ (子基板) / 3 相センシング選択" (at 254 199.3 0) (effects (font (size 1.5 1.5)) (justify left bottom)))
-(property "Sheetfile" "b2b.kicad_sch" (at 254 230.6 0) (effects (font (size 1.27 1.27)) (justify left top)))
+(sheet (at 254 200) (size 70 30) (fields_autoplaced yes) (stroke (width 0.1524) (type solid)) (fill (color 0 0 0 0.0000))
+(property "Sheetname" "DIP 端子 J1/J2 / ゲート確認 LED / センシング選択 / I/O" (at 254 199.3 0) (effects (font (size 1.5 1.5)) (justify left bottom)))
+(property "Sheetfile" "io.kicad_sch" (at 254 230.6 0) (effects (font (size 1.27 1.27)) (justify left top)))
 (instances (project "mPBCH32M030DS0" (path "/87b4cdf7-ae48-57cd-a772-8ad5802448bf" (page "5"))))
 )
-(sheet (at 332 200) (size 70 30) (fields_autoplaced) (stroke (width 0.1524) (type solid)) (fill (color 0 0 0 0.0000))
-(property "Sheetname" "インターフェース (ホール / 通信 / GPIO 引き出し / UI)" (at 332 199.3 0) (effects (font (size 1.5 1.5)) (justify left bottom)))
-(property "Sheetfile" "io.kicad_sch" (at 332 230.6 0) (effects (font (size 1.27 1.27)) (justify left top)))
-(instances (project "mPBCH32M030DS0" (path "/87b4cdf7-ae48-57cd-a772-8ad5802448bf" (page "6"))))
-)
 (sheet_instances (path "/" (page "1")))
