File: hardware/mPBCH32M030DS0.kicad_pcb (KiCad board)
At the start: 2 copper layers, 22.9 x 53.3 mm, 90 parts, among them J1 EDGE_L, J2 EDGE_R, J8 USB-C, SW1 RESET, SW2 USER/BOOT, U1 CH32M030C8U7, U3 USBLC6-2SC6, Y1 8MHz CL=20pF

Commit message: モジュールの nFAULT フィルタ・USB GND 強化, 3D モデルと干渉チェック, 電流容量チェックの道具
- nFAULT (TIM1 BKIN) に 1nF (C120) を追加。470Ω と 0.47µs。CH32M030 の TIM1 には BKIN の
  デジタルフィルタが無いため, ハードの RC で誤停止を防ぐ (配線済みの基板へ追加して迷路配線で接続)
- USB-C (J8) の GND パッド脇に GND ビアを追加し, 下面の GND ベタへ直結 (5A 帰路の細い箇所を解消)
- USB-PD の要求電流を min(want_mA, 3000mA) に頭打ち (J8 の VBUS パッド口元の銅幅で決まる上限)
- KiCad 8 標準に無い 3D モデルを作成 (QFN48 0.35mm, TSON Advance, 1812 / NANO2 ヒューズ)
  tools/gen_3dmodels.py, 割当は gen_pcb.py models
- tools/check_3d.py: STEP で部品どうしの干渉, モジュールを子基板へ挿した状態, ヒートシンク面の高さを確認
- tools/power_check/: 銅箔の抵抗網で電流分布を解き IPC-2221 と比較 / 3.3V 系のノイズ結合の確認
- 下面の部品高さの記述を実測 (3D) の 1.65mm に訂正

Co-Authored-By: Claude Opus 5.5 <noreply@anthropic.com>
Claude-Session: https://claude.ai/code/session_01LENFjjhDfYjJZV1NWhB9uV
Parts:
- added C120: 1nF/50V, C_0402_1005Metric, B.Cu at (10.2, 26.9)
Routing:
- net GND: track 252.5 -> 253.7 mm, vias 17 -> 18
- net nFAULT: track 33.7 -> 34.9 mm
Changed lines of the file:
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@@
 			(zone_connect 2)
 		)
-		(model "${KICAD8_3DMODEL_DIR}/Package_DFN_QFN.3dshapes/QFN-48-1EP_5x5mm_P0.35mm_EP3.7x3.7mm.wrl"
+		(model "${KIPRJMOD}/lib/mPB.3dshapes/QFN-48-1EP_5x5mm_P0.35mm_EP3.7x3.7mm.wrl"
 			(offset
 				(xyz 0 0 0)
@@
 		)
 	)
+	(footprint "C_0402_1005Metric"
+		(layer "B.Cu")
+		(at 10.15 26.93 -90)
+		(descr "Capacitor SMD 0402 (1005 Metric), square (rectangular) end terminal, IPC_7351 nominal, (Body size source: IPC-SM-782 page 76, https://www.pcb-3d.com/wordpress/wp-content/uploads/ipc-sm-782a_amendment_1_and_2.pdf), generated with kicad-footprint-generator")
+		(tags "capacitor")
+		(property "Reference" "C120"
+			(at 0 1.16 90)
+			(layer "B.SilkS")
+			(effects
+				(font
+					(size 0.7 0.7)
+					(thickness 0.1)
+				)
+				(justify mirror)
+			)
+		)
+		(property "Value" "1nF/50V"
+			(at 0 -1.16 90)
+			(layer "B.Fab")
+			(hide yes)
+			(effects
+				(font
+					(size 1 1)
+					(thickness 0.15)
+				)
+				(justify mirror)
+			)
+		)
+		(property "Footprint" ""
+			(at 0 0 90)
+			(unlocked yes)
+			(layer "B.Fab")
+			(hide yes)
+			(effects
+				(font
+					(size 1.27 1.27)
+					(thickness 0.15)
+				)
+				(justify mirror)
+			)
+		)
+		(property "Datasheet" ""
+			(at 0 0 90)
+			(unlocked yes)
+			(layer "B.Fab")
+			(hide yes)
+			(effects
+				(font
+					(size 1.27 1.27)
+					(thickness 0.15)
+				)
+				(justify mirror)
+			)
+		)
+		(property "Description" ""
+			(at 0 0 90)
+			(unlocked yes)
+			(layer "B.Fab")
+			(hide yes)
+			(effects
+				(font
+					(size 1.27 1.27)
+					(thickness 0.15)
+				)
+				(justify mirror)
+			)
+		)
+		(attr smd)
+		(fp_line
+			(start 0.107836 0.36)
+			(end -0.107836 0.36)
+			(stroke
+				(width 0.12)
+				(type solid)
+			)
+			(layer "B.SilkS")
+		)
+		(fp_line
+			(start 0.107836 -0.36)
+			(end -0.107836 -0.36)
+			(stroke
+				(width 0.12)
+				(type solid)
+			)
+			(layer "B.SilkS")
+		)
+		(fp_line
+			(start -0.91 0.46)
+			(end -0.91 -0.46)
+			(stroke
+				(width 0.05)
+				(type solid)
+			)
+			(layer "B.CrtYd")
+		)
+		(fp_line
+			(start 0.91 0.46)
+			(end -0.91 0.46)
+			(stroke
+				(width 0.05)
+				(type solid)
+			)
+			(layer "B.CrtYd")
+		)
+		(fp_line
+			(start -0.91 -0.46)
+			(end 0.91 -0.46)
+			(stroke
+				(width 0.05)
+				(type solid)
+			)
+			(layer "B.CrtYd")
+		)
+		(fp_line
+			(start 0.91 -0.46)
+			(end 0.91 0.46)
+			(stroke
+				(width 0.05)
+				(type solid)
+			)
+			(layer "B.CrtYd")
+		)
+		(fp_line
+			(start -0.5 0.25)
+			(end -0.5 -0.25)
+			(stroke
+				(width 0.1)
+				(type solid)
+			)
+			(layer "B.Fab")
+		)
+		(fp_line
+			(start 0.5 0.25)
+			(end -0.5 0.25)
+			(stroke
+				(width 0.1)
+				(type solid)
+			)
+			(layer "B.Fab")
+		)
+		(fp_line
+			(start -0.5 -0.25)
+			(end 0.5 -0.25)
+			(stroke
+				(width 0.1)
+				(type solid)
+			)
+			(layer "B.Fab")
+		)
+		(fp_line
+			(start 0.5 -0.25)
+			(end 0.5 0.25)
+			(stroke
+				(width 0.1)
+				(type solid)
+			)
+			(layer "B.Fab")
+		)
+		(fp_text user "${REFERENCE}"
+			(at 0 0 90)
+			(layer "B.Fab")
+			(effects
+				(font
+					(size 0.25 0.25)
+					(thickness 0.04)
+				)
+				(justify mirror)
+			)
+		)
+		(pad "1" smd roundrect
+			(at -0.48 0 270)
+			(size 0.56 0.62)
+			(layers "B.Cu" "B.Paste" "B.Mask")
+			(roundrect_rratio 0.25)
+			(net 22 "nFAULT")
+		)
+		(pad "2" smd roundrect
+			(at 0.48 0 270)
+			(size 0.56 0.62)
+			(layers "B.Cu" "B.Paste" "B.Mask")
+			(roundrect_rratio 0.25)
+			(net 5 "GND")
+		)
+		(model "${KICAD8_3DMODEL_DIR}/Capacitor_SMD.3dshapes/C_0402_1005Metric.wrl"
+			(offset
+				(xyz 0 0 0)
+			)
+			(scale
+				(xyz 1 1 1)
+			)
+			(rotate
+				(xyz 0 0 0)
+			)
+		)
+	)
 	(footprint "R_0402_1005Metric"
 		(layer "B.Cu")
@@
 	)
 	(segment
+		(start 16.059999 7.39)
+		(end 16.059999 8.57)
+		(width 0.4)
+		(layer "F.Cu")
+		(net 5)
+	)
+	(segment
 		(start 18.7649 30.3927)
 		(end 18.5283 30.1561)
@@
 	)
 	(via
+		(at 16.059999 8.57)
+		(size 0.6)
+		(drill 0.3)
+		(layers "F.Cu" "B.Cu")
+		(net 5)
+	)
+	(via
 		(at 10.1247 12.9685)
 		(size 0.6)
@@
 	)
 	(segment
+		(start 10.75 27.05)
+		(end 10.75 27.35)
+		(width 0.15)
+		(layer "B.Cu")
+		(net 22)
+	)
+	(segment
 		(start 17.5632 37.6462)
 		(end 16.8244 38.385)
@@
 	)
 	(segment
+		(start 10.35 26.65)
+		(end 10.75 27.05)
+		(width 0.15)
+		(layer "B.Cu")
+		(net 22)
+	)
+	(segment
+		(start 10.75 27.35)
+		(end 10.95 27.55)
+		(width 0.15)
+		(layer "B.Cu")
+		(net 22)
+	)
+	(segment
 		(start 12.4501 29.8019)
 		(end 10.9463 28.2981)
@@
 		(polygon
 			(pts
-				(xy 21.86 1) (xy 21.86 1) (xy 21.86 52.34) (xy 21.86 52.34)
+				(xy 21.86 1) (xy 21.86 52.34)
 			)
 		)
@@
 		(polygon
 			(pts
-				(xy 1 1) (xy 21.86 1) (xy 21.86 1) (xy 1 1)
+				(xy 1 1) (xy 21.86 1)
 			)
 		)
@@
 		(polygon
 			(pts
-				(xy 1 52.34) (xy 21.86 52.34) (xy 21.86 52.34) (xy 1 52.34)
+				(xy 1 52.34) (xy 21.86 52.34)
 			)
 		)
@@
 		(polygon
 			(pts
-				(xy 1 1) (xy 1 1) (xy 1 52.34) (xy 1 52.34)
+				(xy 1 1) (xy 1 52.34)
 			)
 		)

Commit message: MCU モジュール: ピンヘッダを下面実装に (ピンは MCU と反対側), ピン番号を上面シルクに
- J1/J2 を BOTTOM 面へ裏返した (180° 回転 + 反転で 1 番ピンは上端のまま, 穴の位置は不変)。
  ブレッドボード・子基板のソケットに挿しても USB-C とボタンが上を向き, 操作できる
- 上面 (MCU 側) の各ピンの外側にピン番号 1〜21, 下面の信号名は樹脂部の外 (1.5mm) へ
- 配線は確定済みのものをそのまま使う (tools/module_headers_bottom.py)。gen_pcb.py main で作り直す場合も
  配線後に裏返す (flip_after_route)
- DRC: 電気的エラー 0 / 未接続 0。3D: 単体・子基板 A/B に挿した状態とも干渉なし
- 手直し用ベタなし版, 製造データ, パネル, 資料を更新

Co-Authored-By: Claude Opus 5.5 <noreply@anthropic.com>
Claude-Session: https://claude.ai/code/session_01LENFjjhDfYjJZV1NWhB9uV
Parts:
- J1, J2: moved to B.Cu
- turned J1 to 180 degrees
- turned J2 to 180 degrees
Other:
- board text added: "1"
- board text added: "10"
- board text added: "11"
- board text added: "12"
- board text added: "13"
- board text added: "14"
- board text added: "15"
- board text added: "16"
- board text added: "17"
- board text added: "18"
- board text added: "19"
- board text added: "2"
- board text added: "20"
- board text added: "21"
- board text added: "3"
- board text added: "4"
- board text added: "5"
- board text added: "6"
- board text added: "7"
- board text added: "8"
- board text added: "9"
