File: hardware/w9_nopour/mPBCH32M030DS0.kicad_pcb (KiCad board)
At the start: 2 copper layers, 22.9 x 53.3 mm, 90 parts, among them J1 EDGE_L, J2 EDGE_R, J8 USB-C, SW1 RESET, SW2 USER/BOOT, U1 CH32M030C8U7, U3 USBLC6-2SC6, Y1 8MHz CL=20pF

Commit message: 9マス版 MCU モジュールの配線を完成 (未接続 0)
- 水晶 Y1 と C131/C132 を QFN 下辺の XI/XO (8/9 番ピン) 直下の裏面へ移動し、
  下辺ピン 1〜7 の引き出しを空けて再配線 (9 マス版のみ)
- DRC: 未接続 0 / 電気的エラー 0 (シルク警告のみ)
- ベタなし版 (w9_nopour)、製造データ、図、DRC まとめを再生成
- 手配線補助ツール hand_route.py / negot_route.py を追加
- README / stacking.md の状況を更新

Co-Authored-By: Claude Opus 5.5 <noreply@anthropic.com>
Claude-Session: https://claude.ai/code/session_01LENFjjhDfYjJZV1NWhB9uV
Parts:
- Y1: moved to B.Cu
- moved C131 3.94 mm to (12.7, 27.4)
- moved Y1 2.98 mm to (13.5, 24.5), turned to -90 degrees
- moved C132 2.95 mm to (12.7, 28.8)
Routing:
- net IB_N: track 1.45 -> 58.9 mm, vias 0 -> 7
- net I2C_SCL: track 8.11 -> 54.5 mm, vias 0 -> 2
- net IA_P: track 37.3 -> 82.6 mm, vias 3 -> 7
- net IA_N: track 1.45 -> 37.6 mm, vias 0 -> 3
- net nFAULT: track 0.00 -> 33.7 mm, vias 0 -> 4
- net VBUS_SNS: track 57.2 -> 33.8 mm, vias 4 -> 2
- net GPIO_PC4: track 80.5 -> 57.8 mm, vias 3 -> 8
- net I2C_SDA: track 11.2 -> 32.4 mm, vias 0 -> 1
- net GND: track 232.1 -> 252.5 mm, vias 7 -> 12
- net USB_VBUS: track 97.8 -> 78.6 mm, vias 1 -> 0
- net PD_PWR_EN: track 39.8 -> 22.6 mm, vias 1 -> 3
- net +3V3: track 85.9 -> 102.3 mm, vias 6 -> 2
- net QII_IN: track 32.4 -> 17.3 mm
- net OCP_REF: track 41.2 -> 29.5 mm, vias 3 -> 1
- net ISH: track 25.2 -> 14.0 mm, vias 0 -> 2
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