File: hardware/w8_nopour/mPBCH32M030DS0.kicad_pcb (KiCad board)
At the start: 2 copper layers, 20.3 x 53.3 mm, 90 parts, among them J1 EDGE_L, J2 EDGE_R, J8 USB-C, SW1 RESET, SW2 USER/BOOT, U1 CH32M030C8U7, U3 USBLC6-2SC6, Y1 8MHz CL=20pF

Commit message: 8マス版 MCU モジュールの配線を完成 (未接続 0)
- 水晶 Y1 と C131/C132 を XI/XO 直下の裏面へ移す配置を 8 マス版にも適用
- 8 マス版モジュールのみ線幅・間隙 0.10mm / ビア 0.5mm (穴 0.25mm) に詰める
  (0.127mm では 5 通りの試行とも未接続 19〜27 が残ったため)。MPB_RULE / MPB_VIA で上書き可
- DRC: 未接続 0 / 電気的エラー 0 (シルク警告のみ)
- ベタなし版 (w8_nopour)、製造データ、図、DRC まとめを再生成
- README / stacking.md を更新 (両版とも配線完了)

Co-Authored-By: Claude Opus 5.5 <noreply@anthropic.com>
Claude-Session: https://claude.ai/code/session_01LENFjjhDfYjJZV1NWhB9uV
Parts:
- Y1: moved to B.Cu
- moved C132 2.66 mm to (9.97, 28.8)
- moved C131 2.40 mm to (9.97, 27.4)
- moved Y1 1.48 mm to (10.8, 24.5), turned to -90 degrees
Routing:
- net I2C_SCL: track 7.98 -> 70.0 mm, vias 0 -> 8
- net I2C_SDA: track 10.8 -> 57.7 mm, vias 0 -> 2
- net HO3: track 8.96 -> 51.9 mm
- net QII_SRC: track 53.6 -> 18.8 mm, vias 3 -> 1
- net IA_N: track 1.29 -> 32.4 mm, vias 0 -> 3
- net IB_P: track 3.08 -> 33.6 mm, vias 0 -> 1
- net SW2: track 8.99 -> 38.9 mm
- net OCP_REF: track 6.75 -> 36.2 mm, vias 0 -> 1
- net IA_P: track 3.68 -> 31.5 mm, vias 0 -> 1
- net LO2: track 7.73 -> 34.9 mm
- net VHV: track 54.4 -> 80.5 mm, vias 2 -> 4
- net VBUS: track 21.6 -> 46.9 mm, vias 4 -> 3
- net VBUS_SNS: track 7.94 -> 33.2 mm, vias 1 -> 4
- net SENS_W: track 0.00 -> 24.5 mm, vias 0 -> 2
- net nFAULT: track 19.9 -> 44.1 mm, vias 1 -> 4
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