File: hardware/daughter/PWR_A/bridge.kicad_sch (KiCad schematic)
At the start: 76 parts, among them J1 B2B_PWR, J2 OUT0, J3 B2B_SIG, J4 OUT1, J5 OUT2, J6 OUT3, Q1 TPN1R603PL, Q2 TPN1R603PL, Q3 TPN1R603PL, Q4 TPN1R603PL, Q5 TPN1R603PL, Q6 TPN1R603PL, Q7 TPN1R603PL, Q8 TPN1R603PL

Commit message: Rev 0.4: DIP-42 MCU module + power boards A/B/C (KiCad 8)
- MCU module: 20.32 x 53.34mm (8 x 21 grid), DIP-42 (0.6in rows), fits
  an 82 x 52mm breadboard. Headers can be fitted from either side;
  signal names on bottom silk. All LEDs (power, status, 8 gate LEDs) on
  the module top.
- Power boards take the module in two 1x21 sockets (left/right
  symmetric mating). FETs/shunts on the heatsink side, no LEDs.
  Voltage-dependent parts (TVS, OVP divider, bulk caps, BEMF divider)
  moved to the power boards. Breakout board D removed.
  A/C: 20.32 x 71.94mm, B (TO-263 x8): 40.64 x 66.94mm.
- Capacitors re-selected for realistic size vs voltage/capacitance
  (4.7uF 1608, 10uF/25V 2012, 10uF/50V 1206, 4.7nF/100V 1608, low
  profile electrolytics).
- Schematics and boards generated in KiCad 8 format; netlists verified
  with KiCad 8.0.9.
- Layout pipeline: Freerouting bridge (parallel), second pass, early
  repair before pours, island-aware maze repair, DRC via kicad-cli.
- DRC: power boards A/B/C have 0 unconnected / 0 electrical errors.
  The MCU module still has unrouted connections (work in progress).

Co-Authored-By: Claude Opus 5.5 <noreply@anthropic.com>
Claude-Session: https://claude.ai/code/session_01LENFjjhDfYjJZV1NWhB9uV
Parts:
- removed C1, C2: 470uF/25V, Capacitor_THT:CP_Radial_D8.0mm_P3.50mm, symbol mdrv:CP
- removed C30: 0.1uF/50V, Capacitor_SMD:C_0402_1005Metric, symbol mdrv:C
- removed C51: 10uF/50V, Capacitor_SMD:C_0805_2012Metric, symbol mdrv:C
- removed D10: RED GH0, LED_SMD:LED_0603_1608Metric, symbol mdrv:LED
- removed D12: RED GH1, LED_SMD:LED_0603_1608Metric, symbol mdrv:LED
- removed D14: RED GH2, LED_SMD:LED_0603_1608Metric, symbol mdrv:LED
- removed D15: GREEN GL2, LED_SMD:LED_0603_1608Metric, symbol mdrv:LED
- removed D16: RED GH3, LED_SMD:LED_0603_1608Metric, symbol mdrv:LED
- removed D17: GREEN GL3, LED_SMD:LED_0603_1608Metric, symbol mdrv:LED
- removed H1, H2, H3: M2, MountingHole:MountingHole_2.2mm_M2, symbol mdrv:MH
- removed J1: B2B_PWR, Connector_PinSocket_2.54mm:PinSocket_2x05_P2.54mm_Vertical, symbol mdrv:CONN2x5
- removed J2: OUT0, Connector_PinHeader_2.54mm:PinHeader_1x02_P2.54mm_Vertical, symbol mdrv:CONN2
- removed J3: B2B_SIG, Connector_PinSocket_2.54mm:PinSocket_2x11_P2.54mm_Vertical, symbol mdrv:CONN2x11
- removed J4: OUT1, Connector_PinHeader_2.54mm:PinHeader_1x02_P2.54mm_Vertical, symbol mdrv:CONN2
- removed J5: OUT2, Connector_PinHeader_2.54mm:PinHeader_1x02_P2.54mm_Vertical, symbol mdrv:CONN2
- removed J6: OUT3, Connector_PinHeader_2.54mm:PinHeader_1x02_P2.54mm_Vertical, symbol mdrv:CONN2
- removed JP5: ISEL_B, Connector_PinHeader_2.54mm:PinHeader_1x03_P2.54mm_Vertical, symbol mdrv:CONN3
- removed JP7: ISEL_A, Connector_PinHeader_2.54mm:PinHeader_1x03_P2.54mm_Vertical, symbol mdrv:CONN3
- removed R31, R33, R43, R51, R53: 20k, Resistor_SMD:R_0402_1005Metric, symbol mdrv:R
- removed R35, R36, R46, R55, R56, R65, R66: 22k, Resistor_SMD:R_0402_1005Metric, symbol mdrv:R
- removed R42, R50: 47R, Resistor_SMD:R_0402_1005Metric, symbol mdrv:R
- added C40: 0.1uF/50V, Capacitor_SMD:C_0402_1005Metric, symbol mdrv:C
- added J4: MOTOR, Connector_PinHeader_2.54mm:PinHeader_2x08_P2.54mm_Vertical, symbol mdrv:CONN2x8
- added JP5: ISEL_B, Jumper:SolderJumper-3_P1.3mm_Bridged12_RoundedPad1.0x1.5mm_NumberLabels, symbol mdrv:SJ3
- added JP7: ISEL_A, Jumper:SolderJumper-3_P1.3mm_Bridged12_RoundedPad1.0x1.5mm_NumberLabels, symbol mdrv:SJ3
- added Q3: TPN1R603PL, Package_SO:Vishay_PowerPAK_1212-8_Single, symbol mdrv:NMOS
- added R30, R32: 47R, Resistor_SMD:R_0402_1005Metric, symbol mdrv:R
- added R34, R44: 10mR 1% 2W, Resistor_SMD:R_2512_6332Metric, symbol mdrv:R
- C30: renamed from R34; value 10mR 1% 2W -> 0.1uF/50V; footprint Resistor_SMD:R_2512_6332Metric -> Capacitor_SMD:C_0402_1005Metric; symbol mdrv:R -> mdrv:C; MPN 2512 2W (例: Bourns CRA2512-FZ-R010ELF) -> Murata GRM155R71H104KE14D (X7R 1005)
- C31, C41, C61: footprint Capacitor_SMD:C_0805_2012Metric -> Capacitor_SMD:C_1206_3216Metric; MPN TDK C2012X5R1H106K125AC (X5R 2012) ※50V/10uF は 1608 の量産品なし -> Murata GRM31CR61H106KA12L (X5R 1206)
- C51: renamed from D13; value GREEN GL1 -> 10uF/50V; footprint LED_SMD:LED_0603_1608Metric -> Capacitor_SMD:C_1206_3216Metric; symbol mdrv:LED -> mdrv:C; MPN (none) -> Murata GRM31CR61H106KA12L (X5R 1206)
- R31: renamed from R30; value 47R -> 20k
- R33: renamed from R32; value 47R -> 20k
- R42: renamed from D11; value GREEN GL0 -> 47R; footprint LED_SMD:LED_0603_1608Metric -> Resistor_SMD:R_0402_1005Metric; symbol mdrv:LED -> mdrv:R
- R43: renamed from Q3; value TPN1R603PL -> 20k; footprint Package_SO:Vishay_PowerPAK_1212-8_Single -> Resistor_SMD:R_0402_1005Metric; symbol mdrv:NMOS -> mdrv:R; MPN Toshiba TPN1R603PL,L1Q (30V 1.6mΩ Qg 41nC) -> (none)
- R50: renamed from R44; value 10mR 1% 2W -> 47R; footprint Resistor_SMD:R_2512_6332Metric -> Resistor_SMD:R_0402_1005Metric; MPN 2512 2W (例: Bourns CRA2512-FZ-R010ELF) -> (none)
- R51: renamed from C40; value 0.1uF/50V -> 20k; footprint Capacitor_SMD:C_0402_1005Metric -> Resistor_SMD:R_0402_1005Metric; symbol mdrv:C -> mdrv:R; MPN Murata GRM155R71H104KE14D (X7R 1005) -> (none)
- R53: renamed from R45; value 22k -> 20k
Connections:
- net GL1 is gone; now on an unnamed net: Q4.4 (G)
- net HO0: now also R30.1; no longer R31.1
- net HO2: now also R50.1
- net ISA_SEL: now also JP7.2
- net ISB_SEL: now also JP5.2
- net ISH: now also JP7.3, R34.2, R44.2; no longer C30.2, R50.2
- net LO0: now also R32.1; no longer R33.1
- net LO1: now also R42.1
- net SRC0: now also C30.2, R33.2, JP7.1, R34.1; no longer C30.1, R42.1 (K)
- net SRC1: now also R43.2, C40.2, JP5.1, R44.1; no longer C51.1 (K), R50.1, R51.2
- net SRC2: now also C51.2, R53.2, JP5.3
- net SW0: now also R31.2, J4.1 (P1), J4.2 (P2), J4.3 (P3), J4.4 (P4)
- net SW1: now also J4.5 (P5), J4.6 (P6), J4.7 (P7), J4.8 (P8), Q3.1 (S), Q3.2 (S), Q3.3 (S); no longer R43.1 (S), R43.2 (S), R43.3 (S)
- net SW2: now also R51.2, J4.10 (P10), J4.11 (P11), J4.12 (P12), J4.9 (P9)
- net SW3: now also J4.13 (P13), J4.14 (P14), J4.15 (P15), J4.16 (P16)
- net VBUS: now also C30.1, C51.1, C40.1, Q3.5 (D); no longer R43.5 (D), R51.1
- net at R42.2: now also R43.1
- net GH0: no longer names the net of Q1.4 (G)
- net GH0: now also R31.1, R30.2; no longer R31.2
- net GH1: no longer names the net of R40.2, R41.1
- net GH1: now also Q3.4 (G); no longer R43.4 (G), R53.1
- net GH2: no longer names the net of Q5.4 (G)
- net GH2: now also R50.2, R51.1
- net GH3: no longer names the net of Q7.4 (G), R60.2, R61.1
- net GL0: no longer names the net of Q2.4 (G)
- net GL0: now also R33.1, R32.2; no longer R33.2
- net GL2: no longer names the net of Q6.4 (G), R52.2
- net GL2: now also R53.1
- net GL3: no longer names the net of Q8.4 (G), R62.2, R63.1
Other:
- note added: "J4: 1-4=OUT0 5-8=OUT1 9-12=OUT2 13-16=OUT3 (各 4 ピン並列)"
- note added: "R70 は全レッグ共通の帰路 (ISH→GND)。ISH/ISA_SEL/ISB_SEL はシャント端からケルビン配線でソケットへ。"
- note added: "ゲート: 47R 直列 + 20k G-S プルダウン。ゲート確認 LED はモジュール側 (HOx-SWx / LOx-GND)。"
- note added: "バスシャント / 電流チャネル選択 (はんだジャンパ) / モータ出力 J4"
- note added: "分圧 3k 1% / (20k 1% + 3k 1%): 入力電圧上限で ≤ 2.5V。"
- note added: "相電圧 (BEMF) 分圧 / 温度 (NTC)"
- note removed: "J1/J3 は主基板 J9/J10 と同じピン番号で嵌合する (ソケットを 270° 回転して裏面実装, gen_pcb.py で座標検証)。"
- note removed: "JP5 1-2: ISP2=HB1(V相) 2-3: ISP2=HB2(コイルB / DC-B)"
- note removed: "JP7 1-2: ISP1=HB0 (差動) 2-3: ISP1=バス (ISH)"
- note removed: "OUT0-3 (J2/J4/J5/J6): 3相=U/V/W | DC=OUT0-1 (+OUT2-3) | ステッピング=A+,A-,B+,B-"
- note removed: "R70 は全レッグ共通の帰路 (ISH→GND)。ISH/ISA_SEL/ISB_SEL はシャント端からケルビン配線で J3 へ。"
- note removed: "ゲート: 47R 直列 + 20k G-S プルダウン。ゲート確認 LED は G-S 電圧で点灯 (H=赤, L=緑)。"
- note removed: "バスシャント / 電流チャネル選択 (TOP 面) / モータ出力"
- note removed: "分圧 3k 1% / (20k 1% + 3k 1%)。入力電圧上限で ≤ 2.5V になるよう子基板ごとに定数を変える。"
- note removed: "基板間コネクタ (BOTTOM 面, 低背ピンソケット) / バルク容量 / 温度"
- note removed: "相電圧 (BEMF) 分圧 → 主基板 JP2-4 → PA5/PA6/PA7"
- title: mPBCH32M030DS0 Power daughter board A (TPN1R603PL) -> mPBCH32M030DS0 power board A (TPN1R603PL)
- moved on the sheet: R31, R33, R50, R53

Commit message: 子基板 A/C: 電源の銅箔を配線前に置く再レイアウト (A 約4A/相, C 3A)
- レッグを LS/HS の縦ブロックにし, 下面 = ISH の背骨 + SRC/VBUS/SW の島,
  上面 = VBUS の帯と各相 SW の階段状の帯 (J4 は 180° 回転: OUT3 が上)
- 固定ベタは DSN では keepout (縁 0.3mm は同ネットの取り付き用) + via_keepout にして
  自動配線がベタを削らないようにした。2 段配線 (MPB_TWO_PHASE) も用意
- A: ゲート抵抗 (0805) の電極間を SW/GL が抜ける配置 (J2 の並びと FET のゲート位置の上下逆を解消)
- A/C: バルク容量は ISH 戻り (VBUS-ISH), USB 側 TVS (D9) は省略, NTC は下側へ
- 電流チェックに 1mm 平均の密度 (角の電流集中を除く) を追加
- ヒートシンクの干渉チェックは MOSFET の範囲だけに

Co-Authored-By: Claude Opus 5.5 <noreply@anthropic.com>
Claude-Session: https://claude.ai/code/session_01LENFjjhDfYjJZV1NWhB9uV
Parts:
- C31, C41, C51, C61: value 10uF/50V -> 10uF/25V; footprint Capacitor_SMD:C_1206_3216Metric -> Capacitor_SMD:C_0805_2012Metric; MPN Murata GRM31CR61H106KA12L (X5R 1206) -> Murata GRM219R61E106KA12D (X5R 0805, 厚さ 0.85mm)
- R30, R32, R40, R42, R50, R52, R60, R62: footprint Resistor_SMD:R_0402_1005Metric -> Resistor_SMD:R_0805_2012Metric
- R34, R44, R54, R64, R70: value 10mR 1% 2W -> 10mR 1% 0.5W; footprint Resistor_SMD:R_2512_6332Metric -> Resistor_SMD:R_1206_3216Metric; MPN 2512 2W (例: Bourns CRA2512-FZ-R010ELF) -> 1206 0.5W (例: Yageo PE1206FRF7W0R01L)
