File: hardware/daughter/PWR_A/power.kicad_sch (KiCad schematic)
At the start: 22 parts, among them J1 SOCK_L, J2 SOCK_R, J3 PWR_IN, Q10 TPN1R603PL, Q9 TPN2R304PL, U2 78L05, U4 LM74700-Q1, U5 LM74700-Q1

Commit message: Rev 0.4: rework module pinout for routability, power boards regenerated
- Module edge pin order follows the CH32M030 QFN48 pin sides so the
  breakout traces nest instead of crossing (J1: USB_VBUS, PD_PWR_EN,
  PC4/PC5, +3V3, +5V, SWDIO, VBUS, NTC, BEMF, HALL, ISx, TACH;
  J2: RX/TX, nRST, gate drive HO3..LO0, VBUS_SNS, I2C, nFAULT).
- Module: area under the QFN kept for fan-out (filters and the VHV/USB
  diode block moved away, gate LEDs right-aligned to J2).
- Power boards A/B/C re-placed for the new pinout (VBUS divider next to
  J2 VBUS_SNS, LM74700 next to its FET) and re-routed: all three at
  0 unconnected / 0 electrical DRC errors.
- Layout tooling: DRC via kicad-cli in a separate process, reload after
  SES import, selectable Freerouting jar, optional rip-up repair,
  configurable Freerouting timeout.
- MCU module still has unrouted connections (work in progress).

Co-Authored-By: Claude Opus 5.5 <noreply@anthropic.com>
Claude-Session: https://claude.ai/code/session_01LENFjjhDfYjJZV1NWhB9uV
Connections:
- net +5V: now also J1.7 (P7); no longer J1.5 (P5)
- net GPIO_PC4: now also J1.4 (P4); no longer J2.4 (P4)
- net GPIO_PC5: now also J1.5 (P5); no longer J2.5 (P5)
- net HO0: now also J2.14 (P14); no longer J2.15 (P15)
- net HO1: now also J2.11 (P11); no longer J2.12 (P12)
- net HO2: now also J2.8 (P8); no longer J2.9 (P9)
- net HO3: now also J2.5 (P5); no longer J2.6 (P6)
- net I2C_SCL: now also J2.18 (P18); no longer J2.19 (P19)
- net I2C_SDA: now also J2.19 (P19); no longer J2.18 (P18)
- net LO0: now also J2.16 (P16); no longer J2.17 (P17)
- net LO1: now also J2.13 (P13); no longer J2.14 (P14)
- net LO2: now also J2.10 (P10); no longer J2.11 (P11)
- net LO3: now also J2.7 (P7); no longer J2.8 (P8)
- net PD_PWR_EN: now also J1.3 (P3); no longer J1.4 (P4)
- net SW0: now also J2.15 (P15); no longer J2.16 (P16)
- net SW1: now also J2.12 (P12); no longer J2.13 (P13)
- net SW2: now also J2.9 (P9); no longer J2.10 (P10)
- net SW3: now also J2.6 (P6); no longer J2.7 (P7)
- net SWDIO: now also J1.8 (P8); no longer J1.7 (P7)
- net UART_RX: now also J2.2 (P2); no longer J2.3 (P3)
- net UART_TX: now also J2.3 (P3); no longer J2.2 (P2)
- net VBUS_SNS: now also J2.17 (P17); no longer J1.3 (P3)
- net nRST: now also J2.4 (P4); no longer J1.8 (P8)

Commit message: 子基板 A/C: 電源の銅箔を配線前に置く再レイアウト (A 約4A/相, C 3A)
- レッグを LS/HS の縦ブロックにし, 下面 = ISH の背骨 + SRC/VBUS/SW の島,
  上面 = VBUS の帯と各相 SW の階段状の帯 (J4 は 180° 回転: OUT3 が上)
- 固定ベタは DSN では keepout (縁 0.3mm は同ネットの取り付き用) + via_keepout にして
  自動配線がベタを削らないようにした。2 段配線 (MPB_TWO_PHASE) も用意
- A: ゲート抵抗 (0805) の電極間を SW/GL が抜ける配置 (J2 の並びと FET のゲート位置の上下逆を解消)
- A/C: バルク容量は ISH 戻り (VBUS-ISH), USB 側 TVS (D9) は省略, NTC は下側へ
- 電流チェックに 1mm 平均の密度 (角の電流集中を除く) を追加
- ヒートシンクの干渉チェックは MOSFET の範囲だけに

Co-Authored-By: Claude Opus 5.5 <noreply@anthropic.com>
Claude-Session: https://claude.ai/code/session_01LENFjjhDfYjJZV1NWhB9uV
Parts:
- removed C8: 100uF/25V, Capacitor_SMD:CP_Elec_8x6.2, symbol mdrv:CP
- removed D9: SMAJ20A, Diode_SMD:D_SMA, symbol mdrv:D_TVS
- removed U5: LM74700-Q1, Package_TO_SOT_SMD:SOT-23-6, symbol mdrv:LM74700
- added Q10: TPN1R603PL, Package_SO:Vishay_PowerPAK_1212-8_Single, symbol mdrv:NMOS
- C7: value 100uF/25V -> 150uF/25V; MPN Panasonic EEE-FK1E101P (8x6.2mm) -> Panasonic EEE-FK1E151P (8x6.2mm)
- F1: value 10A -> 7A; MPN Littelfuse 0451010.MRL (NANO2 2410, 10A 速断) -> Littelfuse 0451007.MRL (NANO2 2410, 7A 速断)
- U5: renamed from Q10; value TPN1R603PL -> LM74700-Q1; footprint Package_SO:Vishay_PowerPAK_1212-8_Single -> Package_TO_SOT_SMD:SOT-23-6; symbol mdrv:NMOS -> mdrv:LM74700; MPN Toshiba TPN1R603PL,L1Q (USB 側 理想ダイオード) -> TI LM74700QDBVRQ1
Connections:
- net GND: now also U5.2 (GND); no longer C7.2
- net ISH: now also C7.2
- net PD_PWR_EN: now also U5.3 (EN)
- net Q10_G: now also U5.5 (GATE), Q10.4 (G); no longer U5.4 (G)
- net USB_VBUS_P: now also U5.6 (ANODE), Q10.1 (S), Q10.2 (S), Q10.3 (S); no longer U5.1 (S), U5.2 (S), U5.3 (S)
- net VBUS: now also U5.4 (CATHODE), Q10.5 (D); no longer U5.5 (D)
- net VCAP2: now also U5.1 (VCAP)
Other:
- note added: "USB 側 TVS は省略 (A/C: 基板幅の制約)。USB_VBUS_P のサージは Q10 のボディダイオード経由で VBUS のバルク容量が吸収する。"
- note added: "バルク容量の − 側は ISH (バス電流シャント R70 の手前)。レッグの帰路に最短でつなぐ。"
Changed lines of the file:
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@@
 (rectangle (start 150 210) (end 405 285) (stroke (width 0.2) (type dash)) (fill (type none)))
 (text "VBUS 分圧 (OVP / ADC) / ホールセンサ用 5V" (exclude_from_sim no) (at 152 215 0) (effects (font (size 2 2) (thickness 0.3) (bold yes)) (justify left bottom)))
+(text "バルク容量の − 側は ISH (バス電流シャント R70 の手前)。レッグの帰路に最短でつなぐ。" (exclude_from_sim no) (at 153 104 0) (effects (font (size 1.3 1.3)) (justify left bottom)))
 (text "バルク容量はモジュールの真下 (上面, 高さ ≤7mm)。ソケット高 8.5mm の下に収まる。" (exclude_from_sim no) (at 153 110 0) (effects (font (size 1.3 1.3)) (justify left bottom)))
+(text "USB 側 TVS は省略 (A/C: 基板幅の制約)。USB_VBUS_P のサージは Q10 のボディダイオード経由で VBUS のバルク容量が吸収する。" (exclude_from_sim no) (at 153 175 0) (effects (font (size 1.2 1.2)) (justify left bottom)))
 (text "PD_PWR_EN = Low (リセット中も R6 で Low) → OFF。FW が PS_RDY と USB_VBUS_SNS を確認してから ON。" (exclude_from_sim no) (at 153 200 0) (effects (font (size 1.25 1.25)) (justify left bottom)))
 (text "VBUS_SNS → モジュール PB4 (ADC17 + 過電圧リセット 1.5V): OVP 18V (VBUS/12)" (exclude_from_sim no) (at 153 280 0) (effects (font (size 1.25 1.25)) (justify left bottom)))
@@
 (symbol (lib_id "mdrv:FUSE") (at 215 45 90) (unit 1) (exclude_from_sim no) (in_bom yes) (on_board yes) (dnp no)
 (property "Reference" "F1" (at 215 42.2 90) (effects (font (size 1.27 1.27))))
-(property "Value" "10A" (at 215 48.6 90) (effects (font (size 1.27 1.27))))
+(property "Value" "7A" (at 215 48.6 90) (effects (font (size 1.27 1.27))))
 (property "Footprint" "mPB:Fuse_Littelfuse_NANO2_2410" (at 215 45 0) (effects (font (size 1.27 1.27)) (hide yes)))
 (property "Datasheet" "~" (at 215 45 0) (effects (font (size 1.27 1.27)) (hide yes)))
-(property "MPN" "Littelfuse 0451010.MRL (NANO2 2410, 10A 速断)" (at 215 45 0) (effects (font (size 1.27 1.27)) (hide yes)))
+(property "MPN" "Littelfuse 0451007.MRL (NANO2 2410, 7A 速断)" (at 215 45 0) (effects (font (size 1.27 1.27)) (hide yes)))
 (pin "1")
 (pin "2")
@@
 (symbol (lib_id "mdrv:CP") (at 360 60 0) (unit 1) (exclude_from_sim no) (in_bom yes) (on_board yes) (dnp no)
 (property "Reference" "C7" (at 362.54 58.73 0) (effects (font (size 1.27 1.27)) (justify left)))
-(property "Value" "100uF/25V" (at 362.54 61.27 0) (effects (font (size 1.27 1.27)) (justify left)))
+(property "Value" "150uF/25V" (at 362.54 61.27 0) (effects (font (size 1.27 1.27)) (justify left)))
 (property "Footprint" "Capacitor_SMD:CP_Elec_8x6.2" (at 360 60 0) (effects (font (size 1.27 1.27)) (hide yes)))
 (property "Datasheet" "~" (at 360 60 0) (effects (font (size 1.27 1.27)) (hide yes)))
-(property "MPN" "Panasonic EEE-FK1E101P (8x6.2mm)" (at 360 60 0) (effects (font (size 1.27 1.27)) (hide yes)))
+(property "MPN" "Panasonic EEE-FK1E151P (8x6.2mm)" (at 360 60 0) (effects (font (size 1.27 1.27)) (hide yes)))
 (pin "1")
 (pin "2")
@@
 (global_label "VBUS" (shape passive) (at 360 53.65 90) (fields_autoplaced yes) (effects (font (size 1.27 1.27)) (justify left)) (property "Intersheetrefs" "${INTERSHEET_REFS}" (at 360 53.65 0) (effects (font (size 1.27 1.27)) (hide yes))))
 (wire (pts (xy 360 63.81) (xy 360 66.35)) (stroke (width 0) (type default)))
-(global_label "GND" (shape passive) (at 360 66.35 270) (fields_autoplaced yes) (effects (font (size 1.27 1.27)) (justify right)) (property "Intersheetrefs" "${INTERSHEET_REFS}" (at 360 66.35 0) (effects (font (size 1.27 1.27)) (hide yes))))
-(symbol (lib_id "mdrv:CP") (at 375 60 0) (unit 1) (exclude_from_sim no) (in_bom yes) (on_board yes) (dnp no)
-(property "Reference" "C8" (at 377.54 58.73 0) (effects (font (size 1.27 1.27)) (justify left)))
-(property "Value" "100uF/25V" (at 377.54 61.27 0) (effects (font (size 1.27 1.27)) (justify left)))
-(property "Footprint" "Capacitor_SMD:CP_Elec_8x6.2" (at 375 60 0) (effects (font (size 1.27 1.27)) (hide yes)))
-(property "Datasheet" "~" (at 375 60 0) (effects (font (size 1.27 1.27)) (hide yes)))
-(property "MPN" "Panasonic EEE-FK1E101P (8x6.2mm)" (at 375 60 0) (effects (font (size 1.27 1.27)) (hide yes)))
-(pin "1")
-(pin "2")
-(instances (project "mPBCH32M030DS0_PWR_A" (path "/e01e5516-0120-51d1-9602-7aa9be2b05d9/248758b8-9b5f-59d9-8a6b-676ee821fa5f" (reference "C8") (unit 1))))
-)
-(wire (pts (xy 375 56.19) (xy 375 53.65)) (stroke (width 0) (type default)))
-(global_label "VBUS" (shape passive) (at 375 53.65 90) (fields_autoplaced yes) (effects (font (size 1.27 1.27)) (justify left)) (property "Intersheetrefs" "${INTERSHEET_REFS}" (at 375 53.65 0) (effects (font (size 1.27 1.27)) (hide yes))))
-(wire (pts (xy 375 63.81) (xy 375 66.35)) (stroke (width 0) (type default)))
-(global_label "GND" (shape passive) (at 375 66.35 270) (fields_autoplaced yes) (effects (font (size 1.27 1.27)) (justify right)) (property "Intersheetrefs" "${INTERSHEET_REFS}" (at 375 66.35 0) (effects (font (size 1.27 1.27)) (hide yes))))
+(global_label "ISH" (shape passive) (at 360 66.35 270) (fields_autoplaced yes) (effects (font (size 1.27 1.27)) (justify right)) (property "Intersheetrefs" "${INTERSHEET_REFS}" (at 360 66.35 0) (effects (font (size 1.27 1.27)) (hide yes))))
 (symbol (lib_id "mdrv:FUSE") (at 175 150 90) (unit 1) (exclude_from_sim no) (in_bom yes) (on_board yes) (dnp no)
 (property "Reference" "F3" (at 175 147.2 90) (effects (font (size 1.27 1.27))))
@@
 (wire (pts (xy 178.81 150) (xy 181.35 150)) (stroke (width 0) (type default)))
 (label "USB_VBUS_P" (at 181.35 150 0) (fields_autoplaced yes) (effects (font (size 1.27 1.27)) (justify left bottom)))
-(symbol (lib_id "mdrv:D_TVS") (at 200 170 270) (unit 1) (exclude_from_sim no) (in_bom yes) (on_board yes) (dnp no)
-(property "Reference" "D9" (at 202.5 169 90) (effects (font (size 1.27 1.27)) (justify left)))
-(property "Value" "SMAJ20A" (at 202.5 171.5 90) (effects (font (size 1.27 1.27)) (justify left)))
-(property "Footprint" "Diode_SMD:D_SMA" (at 200 170 0) (effects (font (size 1.27 1.27)) (hide yes)))
-(property "Datasheet" "~" (at 200 170 0) (effects (font (size 1.27 1.27)) (hide yes)))
-(property "MPN" "SMAJ20A (USB 側サージ)" (at 200 170 0) (effects (font (size 1.27 1.27)) (hide yes)))
-(pin "1")
-(pin "2")
-(instances (project "mPBCH32M030DS0_PWR_A" (path "/e01e5516-0120-51d1-9602-7aa9be2b05d9/248758b8-9b5f-59d9-8a6b-676ee821fa5f" (reference "D9") (unit 1))))
-)
-(wire (pts (xy 200 166.19) (xy 200 163.65)) (stroke (width 0) (type default)))
-(label "USB_VBUS_P" (at 200 163.65 90) (fields_autoplaced yes) (effects (font (size 1.27 1.27)) (justify left bottom)))
-(wire (pts (xy 200 173.81) (xy 200 176.35)) (stroke (width 0) (type default)))
-(global_label "GND" (shape passive) (at 200 176.35 270) (fields_autoplaced yes) (effects (font (size 1.27 1.27)) (justify right)) (property "Intersheetrefs" "${INTERSHEET_REFS}" (at 200 176.35 0) (effects (font (size 1.27 1.27)) (hide yes))))
 (symbol (lib_id "mdrv:NMOS") (at 250 150 270) (unit 1) (exclude_from_sim no) (in_bom yes) (on_board yes) (dnp no)
 (property "Reference" "Q10" (at 251.27 153.81 0) (effects (font (size 1.27 1.27)) (justify left)))
