File: hardware/daughter/PWR_C/bridge.kicad_sch (KiCad schematic)
At the start: 75 parts, among them J1 B2B_PWR, J2 OUT0, J3 B2B_SIG, J4 OUT1, J5 OUT2, J6 OUT3, Q1 MTN2306AN3, Q2 MTN2306AN3, Q3 MTN2306AN3, Q4 MTN2306AN3, Q5 MTN2306AN3, Q6 MTN2306AN3, Q7 MTN2306AN3, Q8 MTN2306AN3

Commit message: Rev 0.4: DIP-42 MCU module + power boards A/B/C (KiCad 8)
- MCU module: 20.32 x 53.34mm (8 x 21 grid), DIP-42 (0.6in rows), fits
  an 82 x 52mm breadboard. Headers can be fitted from either side;
  signal names on bottom silk. All LEDs (power, status, 8 gate LEDs) on
  the module top.
- Power boards take the module in two 1x21 sockets (left/right
  symmetric mating). FETs/shunts on the heatsink side, no LEDs.
  Voltage-dependent parts (TVS, OVP divider, bulk caps, BEMF divider)
  moved to the power boards. Breakout board D removed.
  A/C: 20.32 x 71.94mm, B (TO-263 x8): 40.64 x 66.94mm.
- Capacitors re-selected for realistic size vs voltage/capacitance
  (4.7uF 1608, 10uF/25V 2012, 10uF/50V 1206, 4.7nF/100V 1608, low
  profile electrolytics).
- Schematics and boards generated in KiCad 8 format; netlists verified
  with KiCad 8.0.9.
- Layout pipeline: Freerouting bridge (parallel), second pass, early
  repair before pours, island-aware maze repair, DRC via kicad-cli.
- DRC: power boards A/B/C have 0 unconnected / 0 electrical errors.
  The MCU module still has unrouted connections (work in progress).

Co-Authored-By: Claude Opus 5.5 <noreply@anthropic.com>
Claude-Session: https://claude.ai/code/session_01LENFjjhDfYjJZV1NWhB9uV
Parts:
- removed C1: 220uF/25V, Capacitor_THT:CP_Radial_D6.3mm_P2.50mm, symbol mdrv:CP
- removed C30, C40: 0.1uF/50V, Capacitor_SMD:C_0402_1005Metric, symbol mdrv:C
- removed D10: RED GH0, LED_SMD:LED_0603_1608Metric, symbol mdrv:LED
- removed D11: GREEN GL0, LED_SMD:LED_0603_1608Metric, symbol mdrv:LED
- removed D12: RED GH1, LED_SMD:LED_0603_1608Metric, symbol mdrv:LED
- removed D13: GREEN GL1, LED_SMD:LED_0603_1608Metric, symbol mdrv:LED
- removed D16: RED GH3, LED_SMD:LED_0603_1608Metric, symbol mdrv:LED
- removed D17: GREEN GL3, LED_SMD:LED_0603_1608Metric, symbol mdrv:LED
- removed H1, H2, H3: M2, MountingHole:MountingHole_2.2mm_M2, symbol mdrv:MH
- removed J1: B2B_PWR, Connector_PinSocket_2.54mm:PinSocket_2x05_P2.54mm_Vertical, symbol mdrv:CONN2x5
- removed J2: OUT0, Connector_PinHeader_2.54mm:PinHeader_1x02_P2.54mm_Vertical, symbol mdrv:CONN2
- removed J3: B2B_SIG, Connector_PinSocket_2.54mm:PinSocket_2x11_P2.54mm_Vertical, symbol mdrv:CONN2x11
- removed J4: OUT1, Connector_PinHeader_2.54mm:PinHeader_1x02_P2.54mm_Vertical, symbol mdrv:CONN2
- removed J5: OUT2, Connector_PinHeader_2.54mm:PinHeader_1x02_P2.54mm_Vertical, symbol mdrv:CONN2
- removed J6: OUT3, Connector_PinHeader_2.54mm:PinHeader_1x02_P2.54mm_Vertical, symbol mdrv:CONN2
- removed JP5: ISEL_B, Connector_PinHeader_2.54mm:PinHeader_1x03_P2.54mm_Vertical, symbol mdrv:CONN3
- removed JP7: ISEL_A, Connector_PinHeader_2.54mm:PinHeader_1x03_P2.54mm_Vertical, symbol mdrv:CONN3
- removed R31, R33: 20k, Resistor_SMD:R_0402_1005Metric, symbol mdrv:R
- removed R35, R36, R45, R46, R55, R56, R65, R66: 22k, Resistor_SMD:R_0402_1005Metric, symbol mdrv:R
- added J4: MOTOR, Connector_PinHeader_2.54mm:PinHeader_2x08_P2.54mm_Vertical, symbol mdrv:CONN2x8
- added R30, R32, R40: 47R, Resistor_SMD:R_0402_1005Metric, symbol mdrv:R
- added R34: 10mR 1% 0.5W, Resistor_SMD:R_1206_3216Metric, symbol mdrv:R
- C30: renamed from R34; value 10mR 1% 0.5W -> 0.1uF/50V; footprint Resistor_SMD:R_1206_3216Metric -> Capacitor_SMD:C_0402_1005Metric; symbol mdrv:R -> mdrv:C; MPN 1206 0.5W (例: Yageo PE1206FRF7W0R01L) -> Murata GRM155R71H104KE14D (X7R 1005)
- C31, C41, C51, C61: footprint Capacitor_SMD:C_0805_2012Metric -> Capacitor_SMD:C_1206_3216Metric; MPN TDK C2012X5R1H106K125AC (X5R 2012) ※50V/10uF は 1608 の量産品なし -> Murata GRM31CR61H106KA12L (X5R 1206)
- C40: renamed from R40; value 47R -> 0.1uF/50V; footprint Resistor_SMD:R_0402_1005Metric -> Capacitor_SMD:C_0402_1005Metric; symbol mdrv:R -> mdrv:C; MPN (none) -> Murata GRM155R71H104KE14D (X7R 1005)
- JP5: renamed from D14; value RED GH2 -> ISEL_B; footprint LED_SMD:LED_0603_1608Metric -> Jumper:SolderJumper-3_P1.3mm_Bridged12_RoundedPad1.0x1.5mm_NumberLabels; symbol mdrv:LED -> mdrv:SJ3; MPN (none) -> はんだジャンパ 3 端子 (1-2 ブリッジ済み: HB1 / 2-3: HB2)
- JP7: renamed from D15; value GREEN GL2 -> ISEL_A; footprint LED_SMD:LED_0603_1608Metric -> Jumper:SolderJumper-3_P1.3mm_Bridged12_RoundedPad1.0x1.5mm_NumberLabels; symbol mdrv:LED -> mdrv:SJ3; MPN (none) -> はんだジャンパ 3 端子 (1-2 ブリッジ済み: HB0 レッグ / 2-3: バス電流)
- R31: renamed from R30; value 47R -> 20k
- R33: renamed from R32; value 47R -> 20k
Connections:
- net HO0: now also R30.1; no longer R31.1
- net HO1: now also R40.1; no longer C40.1
- net ISA_SEL: now also JP7.2
- net ISB_SEL: now also JP5.2
- net ISH: now also JP7.3, R34.2; no longer C30.2
- net LO0: now also R32.1; no longer R33.1
- net SRC0: now also C30.2, JP7.1, R33.2, R34.1; no longer C30.1
- net SRC1: now also C40.2, JP5.1
- net SRC2: now also JP5.3; no longer JP7.1 (K)
- net SW0: now also R31.2, J4.1 (P1), J4.2 (P2), J4.3 (P3), J4.4 (P4)
- net SW1: now also J4.5 (P5), J4.6 (P6), J4.7 (P7), J4.8 (P8)
- net SW2: now also J4.10 (P10), J4.11 (P11), J4.12 (P12), J4.9 (P9); no longer JP5.1 (K)
- net SW3: now also J4.13 (P13), J4.14 (P14), J4.15 (P15), J4.16 (P16)
- net VBUS: now also C30.1, C40.1
- net GH0: no longer names the net of Q1.1 (G)
- net GH0: now also R31.1, R30.2; no longer R31.2
- net GH1: no longer names the net of Q3.1 (G), R41.1
- net GH1: now also R40.2; no longer C40.2
- net GH2: no longer names the net of Q5.1 (G), R50.2, R51.1
- net GH3: no longer names the net of Q7.1 (G), R60.2, R61.1
- net GL0: no longer names the net of Q2.1 (G)
- net GL0: now also R33.1, R32.2; no longer R33.2
- net GL1: no longer names the net of Q4.1 (G), R42.2, R43.1
- net GL2: no longer names the net of Q6.1 (G), R52.2, R53.1
- net GL3: no longer names the net of Q8.1 (G), R62.2, R63.1
Other:
- note added: "J4: 1-4=OUT0 5-8=OUT1 9-12=OUT2 13-16=OUT3 (各 4 ピン並列)"
- note added: "R70 は全レッグ共通の帰路 (ISH→GND)。ISH/ISA_SEL/ISB_SEL はシャント端からケルビン配線でソケットへ。"
- note added: "ゲート: 47R 直列 + 20k G-S プルダウン。ゲート確認 LED はモジュール側 (HOx-SWx / LOx-GND)。"
- note added: "バスシャント / 電流チャネル選択 (はんだジャンパ) / モータ出力 J4"
- note added: "分圧 3k 1% / (20k 1% + 3k 1%): 入力電圧上限で ≤ 2.5V。"
- note added: "相電圧 (BEMF) 分圧 / 温度 (NTC)"
- note removed: "J1/J3 は主基板 J9/J10 と同じピン番号で嵌合する (ソケットを 270° 回転して裏面実装, gen_pcb.py で座標検証)。"
- note removed: "JP5 1-2: ISP2=HB1(V相) 2-3: ISP2=HB2(コイルB / DC-B)"
- note removed: "JP7 1-2: ISP1=HB0 (差動) 2-3: ISP1=バス (ISH)"
- note removed: "OUT0-3 (J2/J4/J5/J6): 3相=U/V/W | DC=OUT0-1 (+OUT2-3) | ステッピング=A+,A-,B+,B-"
- note removed: "R70 は全レッグ共通の帰路 (ISH→GND)。ISH/ISA_SEL/ISB_SEL はシャント端からケルビン配線で J3 へ。"
- note removed: "ゲート: 47R 直列 + 20k G-S プルダウン。ゲート確認 LED は G-S 電圧で点灯 (H=赤, L=緑)。"
- note removed: "バスシャント / 電流チャネル選択 (TOP 面) / モータ出力"
- note removed: "分圧 3k 1% / (20k 1% + 3k 1%)。入力電圧上限で ≤ 2.5V になるよう子基板ごとに定数を変える。"
- note removed: "基板間コネクタ (BOTTOM 面, 低背ピンソケット) / バルク容量 / 温度"
- note removed: "相電圧 (BEMF) 分圧 → 主基板 JP2-4 → PA5/PA6/PA7"
- title: mPBCH32M030DS0 Power daughter board C (MTN2306AN3) -> mPBCH32M030DS0 power board C (MTN2306AN3)
- moved on the sheet: R31, R33

Commit message: 子基板 A/C: 電源の銅箔を配線前に置く再レイアウト (A 約4A/相, C 3A)
- レッグを LS/HS の縦ブロックにし, 下面 = ISH の背骨 + SRC/VBUS/SW の島,
  上面 = VBUS の帯と各相 SW の階段状の帯 (J4 は 180° 回転: OUT3 が上)
- 固定ベタは DSN では keepout (縁 0.3mm は同ネットの取り付き用) + via_keepout にして
  自動配線がベタを削らないようにした。2 段配線 (MPB_TWO_PHASE) も用意
- A: ゲート抵抗 (0805) の電極間を SW/GL が抜ける配置 (J2 の並びと FET のゲート位置の上下逆を解消)
- A/C: バルク容量は ISH 戻り (VBUS-ISH), USB 側 TVS (D9) は省略, NTC は下側へ
- 電流チェックに 1mm 平均の密度 (角の電流集中を除く) を追加
- ヒートシンクの干渉チェックは MOSFET の範囲だけに

Co-Authored-By: Claude Opus 5.5 <noreply@anthropic.com>
Claude-Session: https://claude.ai/code/session_01LENFjjhDfYjJZV1NWhB9uV
Parts:
- C31, C41, C51, C61: value 10uF/50V -> 10uF/25V; footprint Capacitor_SMD:C_1206_3216Metric -> Capacitor_SMD:C_0805_2012Metric; MPN Murata GRM31CR61H106KA12L (X5R 1206) -> Murata GRM219R61E106KA12D (X5R 0805, 厚さ 0.85mm)
Changed lines of the file:
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@@
 (symbol (lib_id "mdrv:C") (at 96.28 71.12 0) (unit 1) (exclude_from_sim no) (in_bom yes) (on_board yes) (dnp no)
 (property "Reference" "C31" (at 98.82 69.85 0) (effects (font (size 1.27 1.27)) (justify left)))
-(property "Value" "10uF/50V" (at 98.82 72.39 0) (effects (font (size 1.27 1.27)) (justify left)))
-(property "Footprint" "Capacitor_SMD:C_1206_3216Metric" (at 96.28 71.12 0) (effects (font (size 1.27 1.27)) (hide yes)))
+(property "Value" "10uF/25V" (at 98.82 72.39 0) (effects (font (size 1.27 1.27)) (justify left)))
+(property "Footprint" "Capacitor_SMD:C_0805_2012Metric" (at 96.28 71.12 0) (effects (font (size 1.27 1.27)) (hide yes)))
 (property "Datasheet" "~" (at 96.28 71.12 0) (effects (font (size 1.27 1.27)) (hide yes)))
-(property "MPN" "Murata GRM31CR61H106KA12L (X5R 1206)" (at 96.28 71.12 0) (effects (font (size 1.27 1.27)) (hide yes)))
+(property "MPN" "Murata GRM219R61E106KA12D (X5R 0805, 厚さ 0.85mm)" (at 96.28 71.12 0) (effects (font (size 1.27 1.27)) (hide yes)))
 (pin "1")
 (pin "2")
@@
 (symbol (lib_id "mdrv:C") (at 194.28 71.12 0) (unit 1) (exclude_from_sim no) (in_bom yes) (on_board yes) (dnp no)
 (property "Reference" "C41" (at 196.82 69.85 0) (effects (font (size 1.27 1.27)) (justify left)))
-(property "Value" "10uF/50V" (at 196.82 72.39 0) (effects (font (size 1.27 1.27)) (justify left)))
-(property "Footprint" "Capacitor_SMD:C_1206_3216Metric" (at 194.28 71.12 0) (effects (font (size 1.27 1.27)) (hide yes)))
+(property "Value" "10uF/25V" (at 196.82 72.39 0) (effects (font (size 1.27 1.27)) (justify left)))
+(property "Footprint" "Capacitor_SMD:C_0805_2012Metric" (at 194.28 71.12 0) (effects (font (size 1.27 1.27)) (hide yes)))
 (property "Datasheet" "~" (at 194.28 71.12 0) (effects (font (size 1.27 1.27)) (hide yes)))
-(property "MPN" "Murata GRM31CR61H106KA12L (X5R 1206)" (at 194.28 71.12 0) (effects (font (size 1.27 1.27)) (hide yes)))
+(property "MPN" "Murata GRM219R61E106KA12D (X5R 0805, 厚さ 0.85mm)" (at 194.28 71.12 0) (effects (font (size 1.27 1.27)) (hide yes)))
 (pin "1")
 (pin "2")
@@
 (symbol (lib_id "mdrv:C") (at 292.28 71.12 0) (unit 1) (exclude_from_sim no) (in_bom yes) (on_board yes) (dnp no)
 (property "Reference" "C51" (at 294.82 69.85 0) (effects (font (size 1.27 1.27)) (justify left)))
-(property "Value" "10uF/50V" (at 294.82 72.39 0) (effects (font (size 1.27 1.27)) (justify left)))
-(property "Footprint" "Capacitor_SMD:C_1206_3216Metric" (at 292.28 71.12 0) (effects (font (size 1.27 1.27)) (hide yes)))
+(property "Value" "10uF/25V" (at 294.82 72.39 0) (effects (font (size 1.27 1.27)) (justify left)))
+(property "Footprint" "Capacitor_SMD:C_0805_2012Metric" (at 292.28 71.12 0) (effects (font (size 1.27 1.27)) (hide yes)))
 (property "Datasheet" "~" (at 292.28 71.12 0) (effects (font (size 1.27 1.27)) (hide yes)))
-(property "MPN" "Murata GRM31CR61H106KA12L (X5R 1206)" (at 292.28 71.12 0) (effects (font (size 1.27 1.27)) (hide yes)))
+(property "MPN" "Murata GRM219R61E106KA12D (X5R 0805, 厚さ 0.85mm)" (at 292.28 71.12 0) (effects (font (size 1.27 1.27)) (hide yes)))
 (pin "1")
 (pin "2")
@@
 (symbol (lib_id "mdrv:C") (at 390.28 71.12 0) (unit 1) (exclude_from_sim no) (in_bom yes) (on_board yes) (dnp no)
 (property "Reference" "C61" (at 392.82 69.85 0) (effects (font (size 1.27 1.27)) (justify left)))
-(property "Value" "10uF/50V" (at 392.82 72.39 0) (effects (font (size 1.27 1.27)) (justify left)))
-(property "Footprint" "Capacitor_SMD:C_1206_3216Metric" (at 390.28 71.12 0) (effects (font (size 1.27 1.27)) (hide yes)))
+(property "Value" "10uF/25V" (at 392.82 72.39 0) (effects (font (size 1.27 1.27)) (justify left)))
+(property "Footprint" "Capacitor_SMD:C_0805_2012Metric" (at 390.28 71.12 0) (effects (font (size 1.27 1.27)) (hide yes)))
 (property "Datasheet" "~" (at 390.28 71.12 0) (effects (font (size 1.27 1.27)) (hide yes)))
-(property "MPN" "Murata GRM31CR61H106KA12L (X5R 1206)" (at 390.28 71.12 0) (effects (font (size 1.27 1.27)) (hide yes)))
-(pin "1")
-(pin "2")
+(property "MPN" "Murata GRM219R61E106KA12D (X5R 0805, 厚さ 0.85mm)" (at 390.28 71.12 0) (effects (font (size 1.27 1.27)) (hide yes)))
+(pin "1")
+(pin "2")
