File: hardware/daughter/PWR_B/power.kicad_sch (KiCad schematic)
At the start: 23 parts, among them J1 SOCK_L, J2 SOCK_R, J3 PWR_IN, Q10 TPN1R603PL, Q9 TPN2R304PL, U2 78L05, U4 LM74700-Q1, U5 LM74700-Q1

Commit message: Rev 0.4: rework module pinout for routability, power boards regenerated
- Module edge pin order follows the CH32M030 QFN48 pin sides so the
  breakout traces nest instead of crossing (J1: USB_VBUS, PD_PWR_EN,
  PC4/PC5, +3V3, +5V, SWDIO, VBUS, NTC, BEMF, HALL, ISx, TACH;
  J2: RX/TX, nRST, gate drive HO3..LO0, VBUS_SNS, I2C, nFAULT).
- Module: area under the QFN kept for fan-out (filters and the VHV/USB
  diode block moved away, gate LEDs right-aligned to J2).
- Power boards A/B/C re-placed for the new pinout (VBUS divider next to
  J2 VBUS_SNS, LM74700 next to its FET) and re-routed: all three at
  0 unconnected / 0 electrical DRC errors.
- Layout tooling: DRC via kicad-cli in a separate process, reload after
  SES import, selectable Freerouting jar, optional rip-up repair,
  configurable Freerouting timeout.
- MCU module still has unrouted connections (work in progress).

Co-Authored-By: Claude Opus 5.5 <noreply@anthropic.com>
Claude-Session: https://claude.ai/code/session_01LENFjjhDfYjJZV1NWhB9uV
Connections:
- net +5V: now also J1.7 (P7); no longer J1.5 (P5)
- net GPIO_PC4: now also J1.4 (P4); no longer J2.4 (P4)
- net GPIO_PC5: now also J1.5 (P5); no longer J2.5 (P5)
- net HO0: now also J2.14 (P14); no longer J2.15 (P15)
- net HO1: now also J2.11 (P11); no longer J2.12 (P12)
- net HO2: now also J2.8 (P8); no longer J2.9 (P9)
- net HO3: now also J2.5 (P5); no longer J2.6 (P6)
- net I2C_SCL: now also J2.18 (P18); no longer J2.19 (P19)
- net I2C_SDA: now also J2.19 (P19); no longer J2.18 (P18)
- net LO0: now also J2.16 (P16); no longer J2.17 (P17)
- net LO1: now also J2.13 (P13); no longer J2.14 (P14)
- net LO2: now also J2.10 (P10); no longer J2.11 (P11)
- net LO3: now also J2.7 (P7); no longer J2.8 (P8)
- net PD_PWR_EN: now also J1.3 (P3); no longer J1.4 (P4)
- net SW0: now also J2.15 (P15); no longer J2.16 (P16)
- net SW1: now also J2.12 (P12); no longer J2.13 (P13)
- net SW2: now also J2.9 (P9); no longer J2.10 (P10)
- net SW3: now also J2.6 (P6); no longer J2.7 (P7)
- net SWDIO: now also J1.8 (P8); no longer J1.7 (P7)
- net UART_RX: now also J2.2 (P2); no longer J2.3 (P3)
- net UART_TX: now also J2.3 (P3); no longer J2.2 (P2)
- net VBUS_SNS: now also J2.17 (P17); no longer J1.3 (P3)
- net nRST: now also J2.4 (P4); no longer J1.8 (P8)

Commit message: 子基板 B を 44.6 x 99.5mm に拡大: M3 丸端子台 x6・ヒートシンク固定穴 x2・電源ベタのはんだ盛り
- 電源 (J3 VIN / J5 GND) と 4 相出力 (J40〜J43) を Würth REDCUBE の M3 丸端子台で受ける
- ヒートシンク固定用 M3 穴 H1/H2。MOSFET・シャントは BOTTOM 面 (ヒートシンク側) に 4 レッグ横並び
- 大電流の銅箔を配線前に固定ベタとして置き, レジスト開口ではんだを盛れるようにした
- 右端の VBUS 帯を表裏 2 層に, レッグ 3 横のネックを裏で迂回, 上端に USB 帰路の GND 帯
- 電流容量 (1 相): 1oz 5.4A / はんだ 0.3mm 7.4A。USB-PD 経路は 3A まで
- D1/C1 の − 側は ISH。面付けパネル (99.94 x 99.76mm), 製造データ, 資料を更新

Co-Authored-By: Claude Opus 5.5 <noreply@anthropic.com>
Claude-Session: https://claude.ai/code/session_01LENFjjhDfYjJZV1NWhB9uV
Parts:
- removed C9: 47uF/35V, Capacitor_SMD:CP_Elec_6.3x5.9, symbol mdrv:CP
- removed D9: SMAJ20A, Diode_SMD:D_SMA, symbol mdrv:D_TVS
- removed F3: 5A, Fuse:Fuse_1812_4532Metric, symbol mdrv:FUSE
- removed J3: PWR_IN, Connector_PinHeader_2.54mm:PinHeader_2x06_P2.54mm_Vertical, symbol mdrv:CONN2x6
- removed Q10: TPN1R603PL, Package_SO:Vishay_PowerPAK_1212-8_Single, symbol mdrv:NMOS
- removed U2: 78L05, Package_TO_SOT_SMD:SOT-89-3, symbol mdrv:REG3
- added C1: 10uF/50V, Capacitor_SMD:C_1206_3216Metric, symbol mdrv:C
- added C5, C6: 0.1uF/50V, Capacitor_SMD:C_0402_1005Metric, symbol mdrv:C
- added C7: 47uF/35V, Capacitor_SMD:CP_Elec_6.3x5.9, symbol mdrv:CP
- added D1: SMBJ24A, Diode_SMD:D_SMB, symbol mdrv:D_TVS
- added J3: VIN, TerminalBlock_Wuerth:Wuerth_REDCUBE-THR_WP-THRBU_74650073_THR, symbol mdrv:TERM1
- added J5: GND, TerminalBlock_Wuerth:Wuerth_REDCUBE-THR_WP-THRBU_74650073_THR, symbol mdrv:TERM1
- C8: renamed from C5; value 0.1uF/50V -> 47uF/35V; footprint Capacitor_SMD:C_0402_1005Metric -> Capacitor_SMD:CP_Elec_6.3x5.9; symbol mdrv:C -> mdrv:CP; MPN Murata GRM155R71H104KE14D (X7R 1005) -> Panasonic EEE-FK1V470P (6.3x6.1mm)
- C9: renamed from D1; value SMBJ24A -> 47uF/35V; footprint Diode_SMD:D_SMB -> Capacitor_SMD:CP_Elec_6.3x5.9; symbol mdrv:D_TVS -> mdrv:CP; MPN SMBJ24A (Vwm 24V) -> Panasonic EEE-FK1V470P (6.3x6.1mm)
- D9: renamed from C7; value 47uF/35V -> SMAJ20A; footprint Capacitor_SMD:CP_Elec_6.3x5.9 -> Diode_SMD:D_SMA; symbol mdrv:CP -> mdrv:D_TVS; MPN Panasonic EEE-FK1V470P (6.3x6.1mm) -> SMAJ20A (USB 側サージ)
- F3: renamed from C1; value 10uF/50V -> 5A; footprint Capacitor_SMD:C_1206_3216Metric -> Fuse:Fuse_1812_4532Metric; symbol mdrv:C -> mdrv:FUSE; MPN Murata GRM31CR61H106KA12L (X5R 1206) -> 1812 5A 速断ヒューズ (例: Bourns SF-1812F500)
- Q10: renamed from C8; value 47uF/35V -> TPN1R603PL; footprint Capacitor_SMD:CP_Elec_6.3x5.9 -> Package_SO:Vishay_PowerPAK_1212-8_Single; symbol mdrv:CP -> mdrv:NMOS; MPN Panasonic EEE-FK1V470P (6.3x6.1mm) -> Toshiba TPN1R603PL,L1Q (USB 側 理想ダイオード)
- U2: renamed from C6; value 0.1uF/50V -> 78L05; footprint Capacitor_SMD:C_0402_1005Metric -> Package_TO_SOT_SMD:SOT-89-3; symbol mdrv:C -> mdrv:REG3; MPN Murata GRM155R71H104KE14D (X7R 1005) -> 78L05 (SOT-89, Vin ≤30V)
Connections:
- net +5V: now also U2.1 (OUT)
- net GND: now also U2.2 (GND), J5.1; no longer C9.2 (A), F3.2, Q10.2
- net ISH: now also C8.2, C9.2, C1.2, C7.2, D1.2 (A)
- net Q10_G: now also Q10.4 (G)
- net USB_VBUS: now also F3.1
- net USB_VBUS_P: now also D9.1 (K), F3.2, Q10.1 (S), Q10.2 (S), Q10.3 (S), C6.2; no longer U2.2
- net VBUS: now also C8.1, Q10.5 (D), U2.3 (IN), C1.1, C7.1, D1.1 (K); no longer D9.1, F3.1, Q10.1
- net VCAP1: now also C5.1; no longer C8.1
- net VCAP2: now also C6.1; no longer U2.1
- net VIN: now also J3.1
- net VIN_F: now also C5.2; no longer C8.2
Other:
- note added: "バルク容量の − 側は ISH (バス電流シャント R70 の手前)。レッグの帰路に最短でつなぐ。"
- moved on the sheet: F3
